File: Building sensor/Designs/EMI_sensor_control_Rev1.0/EMI_sensor_control_Rev1.0.kicad_pcb (KiCad board)
At the start: 4 copper layers, 200 x 100 mm, 212 parts, among them J1 Conn_01x06_Male, J2 Conn_02x07_Odd_Even, J3 DB9_Female, J4 PJ-002AH-SMT-TR, Q1 BSR14, Q2 BSR14, Q3 DMHC3025LSD-13, SW1 SW_SP3T, SW2 SW_Push, U1 LMZM23601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

Commit message: End of Rev 1.01
End of Rev 1.01 change will be made to Rx and Bx connection in 1.02
Parts:
- added R65: R 10k, Resistor_SMD:R_1206_3216Metric_Pad1.42x1.75mm_HandSolder, F.Cu at (172.8, 88.7)
- AE1, AE2, AE3: footprint Connector_Coaxial:SMA_Custom -> Connector_Coaxial:SMA_Molex_73251-2200_Horizontal
- C10, C12, C14, C16, C2, C3, C5, C6, C87, C9, D1, L1, R10, R15, R16, R9, U2, U3, U6: moved to B.Cu
- moved D1 100.9 mm to (172.1, 67.7), turned to 270 degrees
- moved C3 100.0 mm to (164.5, 64.6)
- moved C5 97.2 mm to (159.8, 70.2), turned to 270 degrees
- moved R10 93.9 mm to (168.0, 71.8), turned to 270 degrees
- moved R9 92.8 mm to (168.0, 67.7), turned to 270 degrees
- moved U3 92.4 mm to (164.6, 68.7)
- moved C9 87.5 mm to (163.8, 73.5)
- moved C6 81.9 mm to (170.5, 75.0), turned to 270 degrees
- moved C16 74.5 mm to (161.0, 122.7)
- moved C2 73.0 mm to (162.6, 78.9), turned to 270 degrees
- moved C65 72.1 mm to (100.4, 141.9), turned to 90 degrees
- moved U2 71.5 mm to (166.7, 77.4)
- moved Q1 70.5 mm to (101.8, 70.9), turned to 180 degrees
- moved Q2 69.7 mm to (101.7, 76.6), turned to 180 degrees
- moved C63 68.4 mm to (100.4, 138.3), turned to 90 degrees
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Connections:
- R49 pad 2: SH0 -> SH0r
- U15 pad 45: SH0 -> SH0r
- U9 pad 45: SH0 -> SH0b
Routing:
- net +5V: track 44.8 -> 390.0 mm, vias 3 -> 19
- net VDD1: track 80.2 -> 425.0 mm, vias 17 -> 20
- net +BATT: track 0.00 -> 333.8 mm, vias 0 -> 10
- net ADR0r: track 931.6 -> 1259.8 mm, vias 56 -> 114
- net Pwr1: track 0.00 -> 228.7 mm, vias 0 -> 2
- net -5V: track 32.7 -> 243.3 mm, vias 2 -> 10
- net +2V5: track 18.2 -> 199.9 mm, vias 6 -> 14
- net ADCSync: track 12.4 -> 121.6 mm, vias 2 -> 5
- net DO_Tx: track 0.00 -> 95.5 mm, vias 0 -> 2
- net 5vComm: track 0.00 -> 92.2 mm, vias 0 -> 1
- net DO_Rx: track 0.00 -> 89.8 mm, vias 0 -> 2
- net Vref4.1: track 36.8 -> 120.8 mm, vias 2 -> 5
- net ADCReset: track 4.23 -> 83.1 mm, vias 1 -> 7
- net PWROn: track 0.00 -> 77.4 mm, vias 0 -> 1
- net +1V2: track 3.69 -> 63.4 mm, vias 2 -> 3
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- added copper zone on B.Cu, net BxOut
- added copper zone on B.Cu, net Net-(AE1-Pad2)
Other:
- net class Batt added: clearance 0.2, trace_width 1, via_dia 1.2, via_drill 0.6
- net class Power added: clearance 0.2, trace_width 0.5, via_dia 0.8, via_drill 0.4
- board text added: "3.3 V"
- board text added: "<------ Toward Tx"
- board text added: "Bx"
- board text added: "GND"
- board text added: "JTCK"
- board text added: "JTDI"
- board text added: "JTDO"
- board text added: "JTMS"
- board text added: "JTRST"
- board text added: "NC"
- board text added: "On RC Off"
- board text added: "Pancreas EMI Conductivity Meter Rev 1.01"
- board text added: "Rx"
- board text added: "Torwad Rx/Bx ------>"
- board text added: "Tx"
- board text added: "VCP Rx"
- board text added: "VCP Tx"

Commit message: weekly commit
weekly commit, First of Rev 1.02
Parts:
- removed J1: Conn_01x06_Male, Connector_PinHeader_2.54mm:PinHeader_1x06_P2.54mm_Vertical
- added H1: MountingHole_Pad, MountingHole:MountingHole_2.7mm_M2.5_Pad_Via, F.Cu at (62.1, 54.5)
- added H2: MountingHole_Pad, MountingHole:MountingHole_2.7mm_M2.5_Pad_Via, F.Cu at (252.2, 54.5)
- added H3: MountingHole_Pad, MountingHole:MountingHole_2.7mm_M2.5_Pad_Via, F.Cu at (62.1, 144.5)
- added H4: MountingHole_Pad, MountingHole:MountingHole_2.7mm_M2.5_Pad_Via, F.Cu at (252.2, 144.5)
- J2: footprint Connector_PinHeader_2.54mm:PinHeader_2x07_P2.54mm_Vertical_SMD -> Connector_PinHeader_1.27mm:PinHeader_2x07_P1.27mm_Vertical_SMD
- moved R41 4.31 mm to (244.6, 58.8), turned to 90 degrees
- moved J2 4.26 mm to (121.0, 54.7)
- moved R34 2.99 mm to (231.1, 130.0)
- moved R33 2.97 mm to (242.0, 130.0)
- moved L5 2.89 mm to (240.3, 58.9), turned to 270 degrees
- moved L3 2.00 mm to (238.8, 129.7)
- moved L4 2.00 mm to (234.3, 129.7)
Connections:
- AE2 pad 2: BxOut -> ADR0r
- AE3 pad 1: RxCoilsig- -> RxCoilsig+
- AE3 pad 2: ADR0r -> BxCoilsig
- L3 pad 1: RxCoilsig- -> BxCoilsig
- R33 pad 2: RxCoilsig- -> BxCoilsig
Routing:
- net RxCoilsig-: track 46.2 -> 0.00 mm
- net ADR0r: track 1259.8 -> 1296.2 mm, vias 114 -> 115
- net BxCoilsig: track 60.8 -> 89.5 mm
- net BxOut: track 14.8 -> 0.00 mm
- net RxCoilsig+: track 38.1 -> 28.4 mm
- net JTMS: track 20.5 -> 30.2 mm
- net JTDI: track 32.4 -> 39.5 mm
- net VDD1: track 425.0 -> 431.8 mm
- net JTRST: track 51.5 -> 55.8 mm
- net Net-(L4-Pad1): track 12.0 -> 7.85 mm
- net Net-(L3-Pad2): track 11.8 -> 7.99 mm
- net JTDO: track 45.9 -> 49.6 mm
- net JTCK: track 33.4 -> 35.4 mm
- net Net-(L5-Pad2): track 11.5 -> 10.1 mm
- net VCP_Rx: track 29.7 -> 30.7 mm
- added copper zone on F.Cu, net ADR0r
- added copper zone on B.Cu, net BxCoilsig
- removed copper zone on B.Cu, net BxOut
Other:
- rule solder_mask_min_width: 0.25 -> 0.0889
- board text added: "Pancreas EMI Conductivity Meter Kansas State University Rev 1.02"
- board text removed: "Pancreas EMI Conductivity Meter Rev 1.01"
