File: Building sensor/Designs/EMI_sensor_control_Rev1.0/file5D278C8E.sch (KiCad schematic (older format))
At the start: 12 parts

Commit message: Weekly commit 7/20/2019
Weekly commit 7/20/2019
Parts:
- Q?: symbol dk_Transistors-FETs-MOSFETs-Arrays:DMHC3025LSD-13 -> EMI_sensor_control_Rev1.0-rescue:DMHC3025LSD-13-dk_Transistors-FETs-MOSFETs-Arrays
Changed lines of the file:
@@
 $Descr A4 11693 8268
 encoding utf-8
-Sheet 2 4
+Sheet 2 5
 Title ""
 Date ""
@@
 $EndComp
 $Comp
-L dk_Transistors-FETs-MOSFETs-Arrays:DMHC3025LSD-13 Q?
+L EMI_sensor_control_Rev1.0-rescue:DMHC3025LSD-13-dk_Transistors-FETs-MOSFETs-Arrays Q?
 U 1 1 5D27916E
 P 6050 2750
+AR Path="/5D27916E" Ref="Q?"  Part="1"
+AR Path="/5D278C8F/5D27916E" Ref="Q?"  Part="1"
 F 0 "Q?" H 6278 2647 60  0000 L CNN
 F 1 "DMHC3025LSD-13" H 6278 2753 60  0000 L CNN
@@
 	5600 2950 5650 2950
 $Comp
-L power:+BATT #PWR?
+L power:+BATT #PWR0101
 U 1 1 5D2912BB
 P 4150 2000
-F 0 "#PWR?" H 4150 1850 50  0001 C CNN
+F 0 "#PWR0101" H 4150 1850 50  0001 C CNN
 F 1 "+BATT" H 4165 2173 50  0000 C CNN
 F 2 "" H 4150 2000 50  0001 C CNN
@@
 $EndComp
 $Comp
-L power:+BATT #PWR?
+L power:+BATT #PWR0102
 U 1 1 5D2916C1
 P 4500 3000
-F 0 "#PWR?" H 4500 2850 50  0001 C CNN
+F 0 "#PWR0102" H 4500 2850 50  0001 C CNN
 F 1 "+BATT" H 4515 3173 50  0000 C CNN
 F 2 "" H 4500 3000 50  0001 C CNN
@@
 $EndComp
 $Comp
-L power:+BATT #PWR?
+L power:+BATT #PWR0103
 U 1 1 5D291B91
 P 6050 3350
-F 0 "#PWR?" H 6050 3200 50  0001 C CNN
+F 0 "#PWR0103" H 6050 3200 50  0001 C CNN
 F 1 "+BATT" H 6065 3523 50  0000 C CNN
 F 2 "" H 6050 3350 50  0001 C CNN
@@
 	6050 3150 6050 3350
 $Comp
-L power:GND #PWR?
+L power:GND #PWR0104
 U 1 1 5D292A28
 P 3600 3250
-F 0 "#PWR?" H 3600 3000 50  0001 C CNN
+F 0 "#PWR0104" H 3600 3000 50  0001 C CNN
 F 1 "GND" H 3605 3077 50  0000 C CNN
 F 2 "" H 3600 3250 50  0001 C CNN
@@
 $EndComp
 $Comp
-L power:GND #PWR?
+L power:GND #PWR0105
 U 1 1 5D293605
 P 6400 2250
-F 0 "#PWR?" H 6400 2000 50  0001 C CNN
+F 0 "#PWR0105" H 6400 2000 50  0001 C CNN
 F 1 "GND" H 6405 2077 50  0000 C CNN
 F 2 "" H 6400 2250 50  0001 C CNN
@@
 	6400 2150 6400 2250
 $Comp
-L power:GND #PWR?
+L power:GND #PWR0106
 U 1 1 5D2943BE
 P 3950 4250
-F 0 "#PWR?" H 3950 4000 50  0001 C CNN
+F 0 "#PWR0106" H 3950 4000 50  0001 C CNN
 F 1 "GND" H 3955 4077 50  0000 C CNN
 F 2 "" H 3950 4250 50  0001 C CNN

Commit message: Weekly Push
Weekly Push
Parts:
- gave numbers to parts that had none: 12
Connections:
- net TxC3 is gone; now on net TxC2: R8.2
- net TxC4 is gone; now on net TxC1: R7.2
Other:
- note removed: "1.0\n"
- note removed: "EMI Conductivity Meter Control Ciruit"
- moved on the sheet: AE1, Q1, Q2, Q3, R1, R2, R3, R4, R5, R6, R7, R8

Commit message: Weekly Commit
Weekly Commit 08/09/2019
Parts:
- AE1: footprint (none) -> Connector_Coaxial:SMA_Custom
- Q1, Q2: footprint (none) -> Package_TO_SOT_SMD:SOT-23_Handsoldering
- R1, R2, R3, R4, R5, R6, R7, R8: footprint (none) -> Resistor_SMD:R_0805_2012Metric_Pad1.15x1.40mm_HandSolder
Changed lines of the file:
@@
 F 0 "AE1" H 8730 4114 50  0000 L CNN
 F 1 "Antenna_Loop Tx" H 8730 4023 50  0000 L CNN
-F 2 "" H 8500 4100 50  0001 C CNN
+F 2 "Connector_Coaxial:SMA_Custom" H 8500 4100 50  0001 C CNN
 F 3 "~" H 8500 4100 50  0001 C CNN
 	1    8500 4100
@@
 F 0 "Q1" H 6916 5396 50  0000 L CNN
 F 1 "BSR14" H 6916 5305 50  0000 L CNN
-F 2 "" H 6525 5800 50  0001 C CNN
+F 2 "Package_TO_SOT_SMD:SOT-23_Handsoldering" H 6525 5800 50  0001 C CNN
 F 3 "" H 6525 5800 50  0001 C CNN
 	1    6750 5350
@@
 F 0 "Q2" H 7266 6296 50  0000 L CNN
 F 1 "BSR14" H 7266 6205 50  0000 L CNN
-F 2 "" H 6875 6700 50  0001 C CNN
+F 2 "Package_TO_SOT_SMD:SOT-23_Handsoldering" H 6875 6700 50  0001 C CNN
 F 3 "" H 6875 6700 50  0001 C CNN
 	1    7100 6250
@@
 F 0 "R3" V 7050 5050 50  0000 C CNN
 F 1 "R 1k" V 6934 5050 50  0000 C CNN
-F 2 "" V 6980 5050 50  0001 C CNN
+F 2 "Resistor_SMD:R_0805_2012Metric_Pad1.15x1.40mm_HandSolder" V 6980 5050 50  0001 C CNN
 F 3 "~" H 7050 5050 50  0001 C CNN
 	1    7050 5050
@@
 F 0 "R4" V 7400 4700 50  0000 L CNN
 F 1 "R 4.7k" H 7470 4705 50  0000 L CNN
-F 2 "" V 7330 4750 50  0001 C CNN
+F 2 "Resistor_SMD:R_0805_2012Metric_Pad1.15x1.40mm_HandSolder" V 7330 4750 50  0001 C CNN
 F 3 "~" H 7400 4750 50  0001 C CNN
 	1    7400 4750
@@
 F 0 "R5" V 7400 5950 50  0000 C CNN
 F 1 "R 1k" V 7284 5950 50  0000 C CNN
-F 2 "" V 7330 5950 50  0001 C CNN
+F 2 "Resistor_SMD:R_0805_2012Metric_Pad1.15x1.40mm_HandSolder" V 7330 5950 50  0001 C CNN
 F 3 "~" H 7400 5950 50  0001 C CNN
 	1    7400 5950
@@
 F 0 "R6" V 7750 5700 50  0000 L CNN
 F 1 "R 4.7k" H 7820 5705 50  0000 L CNN
-F 2 "" V 7680 5750 50  0001 C CNN
+F 2 "Resistor_SMD:R_0805_2012Metric_Pad1.15x1.40mm_HandSolder" V 7680 5750 50  0001 C CNN
 F 3 "~" H 7750 5750 50  0001 C CNN
 	1    7750 5750
@@
 F 0 "R1" V 6200 5350 50  0000 C CNN
 F 1 "R 1k" V 6084 5350 50  0000 C CNN
-F 2 "" V 6130 5350 50  0001 C CNN
+F 2 "Resistor_SMD:R_0805_2012Metric_Pad1.15x1.40mm_HandSolder" V 6130 5350 50  0001 C CNN
 F 3 "~" H 6200 5350 50  0001 C CNN
 	1    6200 5350
@@
 F 0 "R2" V 6550 6250 50  0000 C CNN
 F 1 "R 1k" V 6434 6250 50  0000 C CNN
-F 2 "" V 6480 6250 50  0001 C CNN
+F 2 "Resistor_SMD:R_0805_2012Metric_Pad1.15x1.40mm_HandSolder" V 6480 6250 50  0001 C CNN
 F 3 "~" H 6550 6250 50  0001 C CNN
 	1    6550 6250
@@
 F 0 "R8" V 8850 6250 50  0000 L CNN
 F 1 "R 1k" H 8920 6255 50  0000 L CNN
-F 2 "" V 8780 6300 50  0001 C CNN
+F 2 "Resistor_SMD:R_0805_2012Metric_Pad1.15x1.40mm_HandSolder" V 8780 6300 50  0001 C CNN
 F 3 "~" H 8850 6300 50  0001 C CNN
 	1    8850 6300
@@
 F 0 "R7" V 8500 6250 50  0000 L CNN
 F 1 "R 1k" H 8570 6255 50  0000 L CNN
-F 2 "" V 8430 6300 50  0001 C CNN
+F 2 "Resistor_SMD:R_0805_2012Metric_Pad1.15x1.40mm_HandSolder" V 8430 6300 50  0001 C CNN
 F 3 "~" H 8500 6300 50  0001 C CNN
 	1    8500 6300

Commit message: End of Rev 1.01
End of Rev 1.01 change will be made to Rx and Bx connection in 1.02
Parts:
- AE1: footprint Connector_Coaxial:SMA_Custom -> Connector_Coaxial:SMA_Molex_73251-2200_Horizontal
Changed lines of the file:
@@
 F 0 "AE1" H 8730 4114 50  0000 L CNN
 F 1 "Antenna_Loop Tx" H 8730 4023 50  0000 L CNN
-F 2 "Connector_Coaxial:SMA_Custom" H 8500 4100 50  0001 C CNN
+F 2 "Connector_Coaxial:SMA_Molex_73251-2200_Horizontal" H 8500 4100 50  0001 C CNN
 F 3 "~" H 8500 4100 50  0001 C CNN
 	1    8500 4100
