File: Building sensor/Designs/EMI_sensor_control_Rev1.0/file5D3E2E6E.sch (KiCad schematic (older format))
At the start: 40 parts

Commit message: Weekly commit 7/25/19
Weekly commit 7/25/19
Parts:
- removed C? (x10): C 100n, symbol Device:C
- removed C? (x3): C 33p, symbol Device:C
- removed C?: C 10n, symbol Device:C
- removed C?: C 10p, symbol Device:C
- removed C?: C 5.6p, symbol Device:C
- removed FB? (x10): Ferrite_Bead, symbol Device:Ferrite_Bead
- removed L?: L 8.2n, symbol Device:L
- removed R?: R 160k, symbol Device:R
- removed R?: R 10, symbol Device:R
- removed R? (x3): R 1k, symbol Device:R
- removed R? (x2): R 2k, symbol Device:R
- removed R? (x2): R 655, symbol Device:R
- removed R? (x2): R 18, symbol Device:R
- removed U?: AD8021ARZ, R_8, symbol 2019-07-11_16-02-03:AD8021ARZ
- removed U?: AD7763BSVZ, SV_64_2, symbol 2019-07-11_15-43-26:AD7763BSVZ
- added Y?: ECS-3961-400-AU-TR, OSC_ECS-3961-400-AU-TR, symbol ECS-3961-400-AU-TR:ECS-3961-400-AU-TR
Connections:
- net labels added: GNDS, MCLK
- net labels removed: +2V5, +6V, -6V, ADCReset, ADCSync, GNDA, Pin12r, Pin14r, Pin15r, Pin19r, Pin19r+, Pin20r, Pin20r-, Pin21r-, Pin22r+, Pin24r, Pin27r, Pin33r, Pin41r, Pin44r, Pin4r, Pin63r, Pin6r, RxFiltered
- wire segments 209 -> 6

Commit message: Weekly Push
Weekly Push
Parts:
- removed Y?: ECS-3961-400-AU-TR, OSC_ECS-3961-400-AU-TR, symbol ECS-3961-400-AU-TR:ECS-3961-400-AU-TR
Changed lines of the file:
@@
 $Descr A4 11693 8268
 encoding utf-8
-Sheet 5 8
-Title ""
+Sheet 4 9
+Title "Pancreas EMI Conductivity Meter "
 Date ""
-Rev ""
-Comp ""
+Rev "1.01"
+Comp "Kansas State University "
 Comment1 ""
 Comment2 ""
@@
 Comment4 ""
 $EndDescr
-$Sheet
-S 2500 1300 3050 1950
-U 5D43B010
-F0 "ADC Rx" 50
-F1 "file5D43B00F.sch" 50
-$EndSheet
 $Sheet
 S 5800 1300 3050 1950
@@
 F1 "file5D3AC028.sch" 50
 $EndSheet
-$Comp
-L ECS-3961-400-AU-TR:ECS-3961-400-AU-TR Y?
-U 1 1 5D41CD54
-P 7350 4500
-F 0 "Y?" H 7350 4965 50  0000 C CNN
-F 1 "ECS-3961-400-AU-TR" H 7350 4874 50  0000 C CNN
-F 2 "OSC_ECS-3961-400-AU-TR" H 7350 4500 50  0001 L BNN
-F 3 "" H 7350 4500 50  0001 L BNN
-F 4 "XC1904CT-ND" H 7350 4500 50  0001 L BNN "Field4"
-F 5 "SMD-4 ECS International" H 7350 4500 50  0001 L BNN "Field5"
-F 6 "ECS Inc." H 7350 4500 50  0001 L BNN "Field6"
-F 7 "Clock Oscillator 40MHz 5V 30pF 4-Pin SMD T/R" H 7350 4500 50  0001 L BNN "Field7"
-F 8 "https://www.digikey.com/product-detail/en/ecs-inc/ECS-3961-400-AU-TR/XC1904CT-ND/2782029?utm_source=snapeda&utm_medium=aggregator&utm_campaign=symbol" H 7350 4500 50  0001 L BNN "Field8"
-	1    7350 4500
-	1    0    0    -1
-$EndComp
-$Comp
-L power:+5V #PWR?
-U 1 1 5D41D214
-P 6200 4400
-F 0 "#PWR?" H 6200 4250 50  0001 C CNN
-F 1 "+5V" V 6215 4528 50  0000 L CNN
-F 2 "" H 6200 4400 50  0001 C CNN
-F 3 "" H 6200 4400 50  0001 C CNN
-	1    6200 4400
-	0    -1   -1   0
-$EndComp
-$Comp
-L power:GND #PWR?
-U 1 1 5D41D4B7
-P 8350 4950
-F 0 "#PWR?" H 8350 4700 50  0001 C CNN
-F 1 "GND" H 8355 4777 50  0000 C CNN
-F 2 "" H 8350 4950 50  0001 C CNN
-F 3 "" H 8350 4950 50  0001 C CNN
-	1    8350 4950
-	1    0    0    -1
-$EndComp
-Wire Wire Line
-	8150 4800 8350 4800
-Wire Wire Line
-	8350 4800 8350 4950
-Wire Wire Line
-	6550 4400 6200 4400
-$Comp
-L power:GNDS #PWR?
-U 1 1 5D41E4AA
-P 8550 4950
-F 0 "#PWR?" H 8550 4700 50  0001 C CNN
-F 1 "GNDS" H 8555 4777 50  0000 C CNN
-F 2 "" H 8550 4950 50  0001 C CNN
-F 3 "" H 8550 4950 50  0001 C CNN
-	1    8550 4950
-	1    0    0    -1
-$EndComp
-Wire Wire Line
-	8350 4800 8550 4800
-Wire Wire Line
-	8550 4800 8550 4950
-Connection ~ 8350 4800
-Text GLabel 8550 4400 2    50   Input ~ 0
-MCLK
-Wire Wire Line
-	8550 4400 8150 4400
+$Sheet
+S 5800 3550 3050 1950
+U 5DAF1841
+F0 "Receiver Amp and Filter" 50
+F1 "file5DAF1840.sch" 50
+$EndSheet
+$Sheet
+S 2500 1300 3050 1950
+U 5D43B010
+F0 "ADC Rx" 50
+F1 "file5D43B00F.sch" 50
+$EndSheet
 $EndSCHEMATC
