File: Building sensor/Designs/EMI_sensor_control_Rev1.0/file5D43B00F.sch (KiCad schematic (older format))
At the start: 45 parts

Commit message: Weekly Push
Weekly Push
Parts:
- C44, C52, C53, C54, C55, C56, C57, C58, C60, C61: renamed from C?; footprint (none) -> Capacitor_SMD:C_0603_1608Metric_Pad1.05x0.95mm_HandSolder
- C45, C49, C50, C51: renamed from C?; footprint (none) -> Capacitor_SMD:C_0402_1005Metric
- C46: renamed from C?; footprint (none) -> Capacitor_Tantalum_SMD:CP_EIA-7343-30_AVX-N_Pad2.25x2.55mm_HandSolder
- C47, C48: renamed from C?; footprint (none) -> Capacitor_SMD:C_0805_2012Metric_Pad1.15x1.40mm_HandSolder
- C59: renamed from C?; footprint (none) -> Capacitor_SMD:C_0805_2012Metric
- FB11, FB12, FB13, FB14, FB15, FB16, FB17, FB18, FB19, FB20: renamed from FB?; footprint (none) -> Capacitor_SMD:C_0603_1608Metric_Pad1.05x0.95mm_HandSolder
- U14: renamed from U?; footprint R_8 -> (none)
- U15: renamed from U?; footprint SV_64_2 -> (none)
- gave numbers to parts that had none: 15
Connections:
- net GND: now also U15.49 (SCP), U15.58 (*CDIV), U15.60 (SCR)
- net GNDS: now reaches U15.2 (MCLKGND)
- net Vref renamed Vref4.1
Other:
- moved on the sheet: C44, C45, C46, C47, C48, C49, C50, C51, C52, C53, C54, C55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

Commit message: Weekly Commit
Weekly Commit 08/09/2019
Parts:
- C59: footprint Capacitor_SMD:C_0805_2012Metric -> Capacitor_SMD:C_0805_2012Metric_Pad1.15x1.40mm_HandSolder
- L6: footprint (none) -> Inductor_SMD:L_0603_1608Metric_Pad1.05x0.95mm_HandSolder
- R48, R50, R54, R55, R56, R57, R58: footprint (none) -> Resistor_SMD:R_0805_2012Metric_Pad1.15x1.40mm_HandSolder
- R49: value R 5k -> R 10k; footprint (none) -> Resistor_SMD:R_1206_3216Metric_Pad1.42x1.75mm_HandSolder
- R51, R52, R53, R61: footprint (none) -> Resistor_SMD:R_1206_3216Metric_Pad1.42x1.75mm_HandSolder
- R59, R60: value R 655 -> R 649; footprint (none) -> Resistor_SMD:R_0805_2012Metric_Pad1.15x1.40mm_HandSolder
- U14: footprint (none) -> footprints:AD8021ARZ
- U15: footprint (none) -> footprints:AD7763BSVZ
Changed lines of the file:
@@
 $EndDescr
-$Comp
-L 2019-07-11_15-43-26:AD7763BSVZ U15
-U 1 1 5D455FBD
-P 5500 3300
-AR Path="/5D3E2E6F/5D43B010/5D455FBD" Ref="U15"  Part="1"
-AR Path="/5DB20FE4/5D455FBD" Ref="U?"  Part="1"
-F 0 "U15" H 6500 3787 60  0000 C CNN
-F 1 "AD7763BSVZ" H 6500 3681 60  0000 C CNN
-F 2 "" H 6500 3640 60  0001 C CNN
-F 3 "" H 5500 3300 60  0000 C CNN
-	1    5500 3300
-	1    0    0    -1
-$EndComp
 $Comp
 L Device:C C44
@@
 F 0 "R52" V 3950 6100 50  0000 L CNN
 F 1 "R 160k" H 3850 6000 50  0000 L CNN
-F 2 "" V 3880 6150 50  0001 C CNN
+F 2 "Resistor_SMD:R_1206_3216Metric_Pad1.42x1.75mm_HandSolder" V 3880 6150 50  0001 C CNN
 F 3 "~" H 3950 6150 50  0001 C CNN
 	1    3950 6150
@@
 F 0 "C59" H 14300 2700 50  0000 L CNN
 F 1 "C 10n" H 14150 2500 50  0000 L CNN
-F 2 "Capacitor_SMD:C_0805_2012Metric" H 14488 2450 50  0001 C CNN
+F 2 "Capacitor_SMD:C_0805_2012Metric_Pad1.15x1.40mm_HandSolder" H 14488 2450 50  0001 C CNN
 F 3 "~" H 14450 2600 50  0001 C CNN
 	1    14450 2600
@@
 F 0 "R58" V 6350 9850 50  0000 C CNN
 F 1 "R 1k" V 6234 9850 50  0000 C CNN
-F 2 "" V 6280 9850 50  0001 C CNN
+F 2 "Resistor_SMD:R_0805_2012Metric_Pad1.15x1.40mm_HandSolder" V 6280 9850 50  0001 C CNN
 F 3 "~" H 6350 9850 50  0001 C CNN
 	1    6350 9850
@@
 F 0 "R48" V 2550 9750 50  0000 C CNN
 F 1 "R 2k" V 2434 9750 50  0000 C CNN
-F 2 "" V 2480 9750 50  0001 C CNN
+F 2 "Resistor_SMD:R_0805_2012Metric_Pad1.15x1.40mm_HandSolder" V 2480 9750 50  0001 C CNN
 F 3 "~" H 2550 9750 50  0001 C CNN
 	1    2550 9750
@@
 F 0 "R54" V 4450 9150 50  0000 C CNN
 F 1 "R 2k" V 4350 9150 50  0000 C CNN
-F 2 "" V 4380 9150 50  0001 C CNN
+F 2 "Resistor_SMD:R_0805_2012Metric_Pad1.15x1.40mm_HandSolder" V 4380 9150 50  0001 C CNN
 F 3 "~" H 4450 9150 50  0001 C CNN
 	1    4450 9150
@@
 F 0 "R50" V 2850 10150 50  0000 R CNN
 F 1 "R 1k" H 2780 10145 50  0000 R CNN
-F 2 "" V 2780 10100 50  0001 C CNN
+F 2 "Resistor_SMD:R_0805_2012Metric_Pad1.15x1.40mm_HandSolder" V 2780 10100 50  0001 C CNN
 F 3 "~" H 2850 10100 50  0001 C CNN
 	1    2850 10100
@@
 F 0 "U14" H 4500 10037 60  0000 C CNN
 F 1 "AD8021ARZ" H 4500 9931 60  0000 C CNN
-F 2 "" H 4450 9950 60  0001 C CNN
+F 2 "footprints:AD8021ARZ" H 4450 9950 60  0001 C CNN
 F 3 "" H 3350 9750 60  0000 C CNN
 	1    2650 9700
@@
 F 0 "R57" V 6350 9450 50  0000 C CNN
 F 1 "R 1k" V 6234 9450 50  0000 C CNN
-F 2 "" V 6280 9450 50  0001 C CNN
+F 2 "Resistor_SMD:R_0805_2012Metric_Pad1.15x1.40mm_HandSolder" V 6280 9450 50  0001 C CNN
 F 3 "~" H 6350 9450 50  0001 C CNN
 	1    6350 9450
@@
 AR Path="/5DB20FE4/5D4561F0" Ref="R?"  Part="1"
 F 0 "R59" V 7050 9200 50  0000 C CNN
-F 1 "R 655" V 6934 9200 50  0000 C CNN
-F 2 "" V 6980 9200 50  0001 C CNN
+F 1 "R 649" V 6934 9200 50  0000 C CNN
+F 2 "Resistor_SMD:R_0805_2012Metric_Pad1.15x1.40mm_HandSolder" V 6980 9200 50  0001 C CNN
 F 3 "~" H 7050 9200 50  0001 C CNN
 	1    7050 9200
@@
 F 0 "R55" V 5200 4600 50  0000 C CNN
 F 1 "R 18" V 5150 4800 50  0000 C CNN
-F 2 "" V 5130 4600 50  0001 C CNN
+F 2 "Resistor_SMD:R_0805_2012Metric_Pad1.15x1.40mm_HandSolder" V 5130 4600 50  0001 C CNN
 F 3 "~" H 5200 4600 50  0001 C CNN
 	1    5200 4600
@@
 F 0 "R56" V 5200 4700 50  0000 C CNN
 F 1 "R 18" V 5250 4900 50  0000 C CNN
-F 2 "" V 5130 4700 50  0001 C CNN
+F 2 "Resistor_SMD:R_0805_2012Metric_Pad1.15x1.40mm_HandSolder" V 5130 4700 50  0001 C CNN
 F 3 "~" H 5200 4700 50  0001 C CNN
 	1    5200 4700
@@
 F 0 "R51" V 3650 6700 50  0000 C CNN
 F 1 "R 100" V 3534 6700 50  0000 C CNN
-F 2 "" V 3580 6700 50  0001 C CNN
+F 2 "Resistor_SMD:R_1206_3216Metric_Pad1.42x1.75mm_HandSolder" V 3580 6700 50  0001 C CNN
 F 3 "~" H 3650 6700 50  0001 C CNN
 	1    3650 6700
@@
 F 0 "R53" V 4200 6700 50  0000 C CNN
 F 1 "R 10" V 4084 6700 50  0000 C CNN
-F 2 "" V 4130 6700 50  0001 C CNN
+F 2 "Resistor_SMD:R_1206_3216Metric_Pad1.42x1.75mm_HandSolder" V 4130 6700 50  0001 C CNN
 F 3 "~" H 4200 6700 50  0001 C CNN
 	1    4200 6700
@@
 AR Path="/5DB20FE4/5D7C321F" Ref="R?"  Part="1"
 F 0 "R49" V 2850 2250 50  0000 C CNN
-F 1 "R 5k" V 2900 2450 50  0000 C CNN
-F 2 "" V 2780 2250 50  0001 C CNN
+F 1 "R 10k" V 2900 2500 50  0000 C CNN
+F 2 "Resistor_SMD:R_1206_3216Metric_Pad1.42x1.75mm_HandSolder" V 2780 2250 50  0001 C CNN
 F 3 "~" H 2850 2250 50  0001 C CNN
 	1    2850 2250
@@
 F 0 "R61" V 14450 2050 50  0000 L CNN
 F 1 "R 10" H 14520 2055 50  0000 L CNN
-F 2 "" V 14380 2100 50  0001 C CNN
+F 2 "Resistor_SMD:R_1206_3216Metric_Pad1.42x1.75mm_HandSolder" V 14380 2100 50  0001 C CNN
 F 3 "~" H 14450 2100 50  0001 C CNN
 	1    14450 2100
@@
 F 0 "L6" V 11850 2100 50  0000 C CNN
 F 1 "L 8.2n" V 11900 1950 50  0000 C CNN
-F 2 "" H 11800 1950 50  0001 C CNN
+F 2 "Inductor_SMD:L_0603_1608Metric_Pad1.05x0.95mm_HandSolder" H 11800 1950 50  0001 C CNN
 F 3 "~" H 11800 1950 50  0001 C CNN
 	1    11800 1950
@@
 AR Path="/5DB20FE4/5D4561EA" Ref="R?"  Part="1"
 F 0 "R60" V 7050 10150 50  0000 C CNN
-F 1 "R 655" V 6934 10150 50  0000 C CNN
-F 2 "" V 6980 10150 50  0001 C CNN
+F 1 "R 649" V 6934 10150 50  0000 C CNN
+F 2 "Resistor_SMD:R_0805_2012Metric_Pad1.15x1.40mm_HandSolder" V 6980 10150 50  0001 C CNN
 F 3 "~" H 7050 10150 50  0001 C CNN
 	1    7050 10150
 	0    1    1    0
 $EndComp
+$Comp
+L 2019-07-11_15-43-26:AD7763BSVZ U15
+U 1 1 5D4E2371
+P 5500 3300
+F 0 "U15" H 6500 3787 60  0000 C CNN
+F 1 "AD7763BSVZ" H 6500 3681 60  0000 C CNN
+F 2 "footprints:AD7763BSVZ" H 6500 3640 60  0001 C CNN
+F 3 "" H 5500 3300 60  0000 C CNN
+	1    5500 3300
+	1    0    0    -1
+$EndComp
 $EndSCHEMATC

Commit message: End of Rev 1.01
End of Rev 1.01 change will be made to Rx and Bx connection in 1.02
Connections:
- net SH0 renamed SH0r
Changed lines of the file:
@@
 SH1
 Text GLabel 3100 2250 2    50   Input ~ 0
-SH0
+SH0r
 Wire Wire Line
 	3100 2250 3000 2250
@@
 SH1
 Text GLabel 8100 5600 2    50   Input ~ 0
-SH0
+SH0r
 Wire Wire Line
 	8100 5900 7500 5900
