File: Building sensor/Designs/EMI_sensor_control_Rev1.0/file5D43B07A.sch (KiCad schematic (older format))
At the start: 46 parts

Commit message: Weekly Push
Weekly Push
Parts:
- removed C? (x10): C 100n, symbol Device:C
- removed C? (x3): C 33p, symbol Device:C
- removed C? (x2): C 10n, symbol Device:C
- removed C?: C 10p, symbol Device:C
- removed C?: C 5.6p, symbol Device:C
- removed C?: C 100u, symbol Device:C
- removed FB? (x10): Ferrite_Bead, symbol Device:Ferrite_Bead
- removed L?: L 8.2n, symbol Device:L
- removed R?: R 160k, symbol Device:R
- removed R? (x2): R 10, symbol Device:R
- removed R? (x3): R 1k, symbol Device:R
- removed R? (x2): R 2k, symbol Device:R
- removed R? (x2): R 655, symbol Device:R
- removed R? (x2): R 18, symbol Device:R
- removed R?: R 100, symbol Device:R
- removed R?: R 5k, symbol Device:R
- removed U?: AD7763BSVZ, SV_64_2, symbol 2019-07-11_15-43-26:AD7763BSVZ
- removed U?: AD8021ARZ, R_8, symbol 2019-07-11_16-02-03:AD8021ARZ
- added C17, C25, C26, C27, C28, C29, C30, C31, C33, C34: C 100n, Capacitor_SMD:C_0603_1608Metric_Pad1.05x0.95mm_HandSolder, symbol Device:C
- added C18, C23, C24: C 33p, Capacitor_SMD:C_0402_1005Metric, symbol Device:C
- added C19: C 100u, Capacitor_Tantalum_SMD:CP_EIA-7343-30_AVX-N_Pad2.25x2.55mm_HandSolder, symbol Device:C
- added C20: C 10p, Capacitor_SMD:C_0805_2012Metric_Pad1.15x1.40mm_HandSolder, symbol Device:C
- added C21, C32: C 10n, Capacitor_SMD:C_0805_2012Metric_Pad1.15x1.40mm_HandSolder, symbol Device:C
- added C22: C 5.6p, Capacitor_SMD:C_0402_1005Metric, symbol Device:C
- added FB1, FB10, FB2, FB3, FB4, FB5, FB6, FB7, FB8, FB9: Ferrite_Bead, Capacitor_SMD:C_0603_1608Metric_Pad1.05x0.95mm_HandSolder, symbol Device:Ferrite_Bead
- added L2: L 8.2n, symbol Device:L
- added R17, R23: R 2k, symbol Device:R
- added R19, R26, R27: R 1k, symbol Device:R
- added R20: R 100, symbol Device:R
- added R21: R 160k, symbol Device:R
- added R22, R30: R 10, symbol Device:R
- added R24, R25: R 18, symbol Device:R
- added R28, R29: R 655, symbol Device:R
- added U8: AD8021ARZ, symbol 2019-07-11_16-02-03:AD8021ARZ
- added U9: AD7763BSVZ, symbol 2019-07-11_15-43-26:AD7763BSVZ
- gave numbers to parts that had none: 1
Connections:
- net +2V5: now also FB10.1, FB2.1, FB3.1, FB5.1, FB6.1
- net +5V: now also FB1.1, FB4.1, FB7.1, FB8.1, FB9.1, U8.7 (+VS), U8.8 (DISABLE*)
- net -5V: now also C20.2, U8.4 (-VS)
- net ADCReset: now also U9.37 (*RESET)
- net ADCSync: now also U9.36 (*SYNC)
- net ADR0b: now also U9.48 (ADR0)
- net BxFiltered: now also R17.2, R26.2
- net DRDY: now also U9.38 (*DRDY)
- net FSI: now also U9.51 (*FSI)
- net FSOb: now also U9.56 (*FSO)
- net GND: now also C17.2, C18.2, C19.2, C21.2, C25.2, C26.2, C27.2, C28.2, C29.2, C30.2, C31.2, C32.2, C33.2, C34.2, R19.1, R21.2, U8.1 (LOGIC_REFERENCE), U9.1 (DGND), U9.11 (AGND4), U9.13 (AGND2), U9.16 (AGND2), U9.18 (AGND2), U9.23 (AGND3), U9.28 (AGND2), U9.29 (AGND3), U9.31 (AGND3), U9.32 (AGND3), U9.34 (AGND1), U9.35 (DGND), U9.42 (DGND), U9.43 (DGND), U9.46 (ADR2), U9.47 (ADR1), U9.49 (SCP), U9.5 (AGND2), U9.53 (DGND), U9.57 (DGND), U9.58 (*CDIV), U9.59 (DGND), U9.60 (SCR), U9.61 (I2C), U9.62 (DGND), U9.64 (DGND), U9.7 (AGND1), U9.EP
- net GNDREF: now also U9.9 (REFGND)
- net MCLK: now also U9.3 (MCLK)
- net Pin12b: now also FB8.2, R30.1, U9.12 (AVDD4)
- net Pin14b: now also C31.1, FB7.2, L2.2, U9.14 (AVDD2)
- net Pin15b: now also C28.1, FB4.2, U9.15 (AVDD2)
- net Pin19b: now also C22.1, C23.2, R26.1, R28.2, U9.19 (VINA+)
- net Pin20b: now also C22.2, C24.2, R27.1, R29.2, U9.20 (VINA-)
- net Pin21b-: now also C23.1, R25.2, R28.1, U9.21 (VOUTA-)
- net Pin22b+: now also C24.1, R24.2, R29.1, U9.22 (VOUTA+)
- net Pin24b: now also C33.1, FB9.2, U9.24 (AVDD3)
- net Pin27b: now also L2.1, U9.27 (AVDD2)
- net Pin33b: now also C29.1, FB5.2, U9.33 (AVDD1)
- net Pin41b: now also C34.1, FB10.2, U9.41 (DVDD)
- net Pin44b: now also C27.1, FB3.2, U9.44 (VDRIVE)
- net Pin4b: now also C25.1, FB1.2, U9.4 (AVDD2)
- net Pin63b: now also C30.1, FB6.2, U9.63 (VDRIVE)
- net Pin6b: now also C26.1, FB2.2, U9.6 (AVDD1)
- net SDI: now also U9.52 (SDI)
- net SDLb: now also U9.50 (SDL)
- net SDO: now also U9.54 (SDO)
- net SH0: now also U9.45 (SH0)
- new net: C21.1, R22.1, U9.10 (VREF+)
- new net: R21.1, U9.17 (RBIAS)
- new net: R25.1, U9.25 (VIN+)
- new net: R24.1, U9.26 (VIN-)
- new net: C18.1, U9.30 (DECAPB)
- new net: C17.1, U9.8 (DECAPA)
- new net: C32.1, R30.2
- new net: R23.1, R27.2, U8.6 (VOUT)
- new net: R17.1, R23.2, U8.2 (-IN)
- new net: R19.2, U8.3 (+IN)
- new net: C20.1, U8.5 (CCOMP)
- new net: C19.1, R20.1, R22.2
- new net GNDS: U9.2 (MCLKGND)
- new net SCO: U9.55 (SCO)
- new net SH1: U9.40 (SH1)
- new net SH2: U9.39 (SH2)
- new net Vref4.1: R20.2
Other:
- moved on the sheet: R18

Commit message: Weekly Commit
Weekly Commit 08/09/2019
Parts:
- L2: footprint (none) -> Inductor_SMD:L_0603_1608Metric_Pad1.05x0.95mm_HandSolder
- R17, R19, R23, R24, R25, R26, R27: footprint (none) -> Resistor_SMD:R_0805_2012Metric_Pad1.15x1.40mm_HandSolder
- R18: value R 5k -> R 10k; footprint (none) -> Resistor_SMD:R_1206_3216Metric_Pad1.42x1.75mm_HandSolder
- R20, R21, R22, R30: footprint (none) -> Resistor_SMD:R_1206_3216Metric_Pad1.42x1.75mm_HandSolder
- R28, R29: value R 655 -> R 649; footprint (none) -> Resistor_SMD:R_0805_2012Metric_Pad1.15x1.40mm_HandSolder
- U8: footprint (none) -> footprints:AD8021ARZ
- U9: footprint (none) -> footprints:AD7763BSVZ
Changed lines of the file:
@@
 AR Path="/5D3E2E6F/5D43B07B/5DB15B2C" Ref="R18"  Part="1"
 F 0 "R18" V 2850 2650 50  0000 C CNN
-F 1 "R 5k" V 2900 2850 50  0000 C CNN
-F 2 "" V 2780 2650 50  0001 C CNN
+F 1 "R 10k" V 2900 2900 50  0000 C CNN
+F 2 "Resistor_SMD:R_1206_3216Metric_Pad1.42x1.75mm_HandSolder" V 2780 2650 50  0001 C CNN
 F 3 "~" H 2850 2650 50  0001 C CNN
 	1    2850 2650
@@
 Text GLabel 8100 6450 2    50   Input ~ 0
 SCO
-$Comp
-L 2019-07-11_15-43-26:AD7763BSVZ U?
-U 1 1 5D8AD58F
-P 5500 3250
-AR Path="/5D3E2E6F/5D43B010/5D8AD58F" Ref="U?"  Part="1"
-AR Path="/5DB20FE4/5D8AD58F" Ref="U?"  Part="1"
-AR Path="/5D3E2E6F/5D43B07B/5D8AD58F" Ref="U9"  Part="1"
-F 0 "U9" H 6500 3737 60  0000 C CNN
-F 1 "AD7763BSVZ" H 6500 3631 60  0000 C CNN
-F 2 "" H 6500 3590 60  0001 C CNN
-F 3 "" H 5500 3250 60  0000 C CNN
-	1    5500 3250
-	1    0    0    -1
-$EndComp
 $Comp
 L Device:C C?
@@
 F 0 "R21" V 3950 6050 50  0000 L CNN
 F 1 "R 160k" H 3650 5950 50  0000 L CNN
-F 2 "" V 3880 6100 50  0001 C CNN
+F 2 "Resistor_SMD:R_1206_3216Metric_Pad1.42x1.75mm_HandSolder" V 3880 6100 50  0001 C CNN
 F 3 "~" H 3950 6100 50  0001 C CNN
 	1    3950 6100
@@
 F 0 "R30" V 14450 2000 50  0000 L CNN
 F 1 "R 10" H 14520 2005 50  0000 L CNN
-F 2 "" V 14380 2050 50  0001 C CNN
+F 2 "Resistor_SMD:R_1206_3216Metric_Pad1.42x1.75mm_HandSolder" V 14380 2050 50  0001 C CNN
 F 3 "~" H 14450 2050 50  0001 C CNN
 	1    14450 2050
@@
 F 0 "L2" V 11850 2050 50  0000 C CNN
 F 1 "L 8.2n" V 11900 1900 50  0000 C CNN
-F 2 "" H 11800 1900 50  0001 C CNN
+F 2 "Inductor_SMD:L_0603_1608Metric_Pad1.05x0.95mm_HandSolder" H 11800 1900 50  0001 C CNN
 F 3 "~" H 11800 1900 50  0001 C CNN
 	1    11800 1900
@@
 F 0 "R27" V 6350 9800 50  0000 C CNN
 F 1 "R 1k" V 6234 9800 50  0000 C CNN
-F 2 "" V 6280 9800 50  0001 C CNN
+F 2 "Resistor_SMD:R_0805_2012Metric_Pad1.15x1.40mm_HandSolder" V 6280 9800 50  0001 C CNN
 F 3 "~" H 6350 9800 50  0001 C CNN
 	1    6350 9800
@@
 F 0 "R17" V 2550 9700 50  0000 C CNN
 F 1 "R 2k" V 2434 9700 50  0000 C CNN
-F 2 "" V 2480 9700 50  0001 C CNN
+F 2 "Resistor_SMD:R_0805_2012Metric_Pad1.15x1.40mm_HandSolder" V 2480 9700 50  0001 C CNN
 F 3 "~" H 2550 9700 50  0001 C CNN
 	1    2550 9700
@@
 F 0 "R23" V 4450 9100 50  0000 C CNN
 F 1 "R 2k" V 4334 9100 50  0000 C CNN
-F 2 "" V 4380 9100 50  0001 C CNN
+F 2 "Resistor_SMD:R_0805_2012Metric_Pad1.15x1.40mm_HandSolder" V 4380 9100 50  0001 C CNN
 F 3 "~" H 4450 9100 50  0001 C CNN
 	1    4450 9100
@@
 F 0 "R19" V 2850 10100 50  0000 R CNN
 F 1 "R 1k" H 2780 10095 50  0000 R CNN
-F 2 "" V 2780 10050 50  0001 C CNN
+F 2 "Resistor_SMD:R_0805_2012Metric_Pad1.15x1.40mm_HandSolder" V 2780 10050 50  0001 C CNN
 F 3 "~" H 2850 10050 50  0001 C CNN
 	1    2850 10050
@@
 F 0 "U8" H 4500 9987 60  0000 C CNN
 F 1 "AD8021ARZ" H 4500 9881 60  0000 C CNN
-F 2 "" H 4450 9900 60  0001 C CNN
+F 2 "footprints:AD8021ARZ" H 4450 9900 60  0001 C CNN
 F 3 "" H 3350 9700 60  0000 C CNN
 	1    2650 9650
@@
 F 0 "R26" V 6350 9400 50  0000 C CNN
 F 1 "R 1k" V 6234 9400 50  0000 C CNN
-F 2 "" V 6280 9400 50  0001 C CNN
+F 2 "Resistor_SMD:R_0805_2012Metric_Pad1.15x1.40mm_HandSolder" V 6280 9400 50  0001 C CNN
 F 3 "~" H 6350 9400 50  0001 C CNN
 	1    6350 9400
@@
 AR Path="/5D3E2E6F/5D43B07B/5D8AD74A" Ref="R29"  Part="1"
 F 0 "R29" V 7050 10100 50  0000 C CNN
-F 1 "R 655" V 6934 10100 50  0000 C CNN
-F 2 "" V 6980 10100 50  0001 C CNN
+F 1 "R 649" V 6934 10100 50  0000 C CNN
+F 2 "Resistor_SMD:R_0805_2012Metric_Pad1.15x1.40mm_HandSolder" V 6980 10100 50  0001 C CNN
 F 3 "~" H 7050 10100 50  0001 C CNN
 	1    7050 10100
@@
 AR Path="/5D3E2E6F/5D43B07B/5D8AD750" Ref="R28"  Part="1"
 F 0 "R28" V 7050 9150 50  0000 C CNN
-F 1 "R 655" V 6934 9150 50  0000 C CNN
-F 2 "" V 6980 9150 50  0001 C CNN
+F 1 "R 649" V 6934 9150 50  0000 C CNN
+F 2 "Resistor_SMD:R_0805_2012Metric_Pad1.15x1.40mm_HandSolder" V 6980 9150 50  0001 C CNN
 F 3 "~" H 7050 9150 50  0001 C CNN
 	1    7050 9150
@@
 F 0 "R24" V 5200 4550 50  0000 C CNN
 F 1 "R 18" V 5150 4800 50  0000 C CNN
-F 2 "" V 5130 4550 50  0001 C CNN
+F 2 "Resistor_SMD:R_0805_2012Metric_Pad1.15x1.40mm_HandSolder" V 5130 4550 50  0001 C CNN
 F 3 "~" H 5200 4550 50  0001 C CNN
 	1    5200 4550
@@
 F 0 "R25" V 5200 4650 50  0000 C CNN
 F 1 "R 18" V 5250 4900 50  0000 C CNN
-F 2 "" V 5130 4650 50  0001 C CNN
+F 2 "Resistor_SMD:R_0805_2012Metric_Pad1.15x1.40mm_HandSolder" V 5130 4650 50  0001 C CNN
 F 3 "~" H 5200 4650 50  0001 C CNN
 	1    5200 4650
@@
 F 0 "R20" V 3650 6650 50  0000 C CNN
 F 1 "R 100" V 3534 6650 50  0000 C CNN
-F 2 "" V 3580 6650 50  0001 C CNN
+F 2 "Resistor_SMD:R_1206_3216Metric_Pad1.42x1.75mm_HandSolder" V 3580 6650 50  0001 C CNN
 F 3 "~" H 3650 6650 50  0001 C CNN
 	1    3650 6650
@@
 F 0 "R22" V 4200 6650 50  0000 C CNN
 F 1 "R 10" V 4084 6650 50  0000 C CNN
-F 2 "" V 4130 6650 50  0001 C CNN
+F 2 "Resistor_SMD:R_1206_3216Metric_Pad1.42x1.75mm_HandSolder" V 4130 6650 50  0001 C CNN
 F 3 "~" H 4200 6650 50  0001 C CNN
 	1    4200 6650
@@
 Wire Wire Line
 	3950 5850 5500 5850
-Wire Wire Line
-	3550 5450 5500 5450
-Wire Wire Line
-	3250 5350 5500 5350
 $Comp
 L power:+2V5 #PWR?
@@
 	2250 2950 2350 2950
 Connection ~ 2350 2950
+$Comp
+L 2019-07-11_15-43-26:AD7763BSVZ U9
+U 1 1 5D4D98BD
+P 5500 3250
+F 0 "U9" H 6500 3737 60  0000 C CNN
+F 1 "AD7763BSVZ" H 6500 3631 60  0000 C CNN
+F 2 "footprints:AD7763BSVZ" H 6500 3590 60  0001 C CNN
+F 3 "" H 5500 3250 60  0000 C CNN
+	1    5500 3250
+	1    0    0    -1
+$EndComp
+Wire Wire Line
+	3550 5450 5500 5450
+Wire Wire Line
+	3250 5350 5500 5350
 $EndSCHEMATC

Commit message: End of Rev 1.01
End of Rev 1.01 change will be made to Rx and Bx connection in 1.02
Parts:
- added R65: R 10k, Resistor_SMD:R_1206_3216Metric_Pad1.42x1.75mm_HandSolder, symbol Device:R
Connections:
- net +2V5: now also R65.1
- net SH0 renamed SH0b
- net SH0b: now also R65.2
Changed lines of the file:
@@
 ADR0b
 Text GLabel 8100 5550 2    50   Input ~ 0
-SH0
+SH0b
 Text GLabel 8100 6350 2    50   Input ~ 0
 SDO
@@
 	3000 2650 3100 2650
 Wire Wire Line
-	2700 2650 2250 2650
+	2700 2650 2350 2650
 Text GLabel 5250 5050 0    50   Input ~ 0
 Pin20b
@@
 Wire Wire Line
 	3250 5350 5500 5350
+$Comp
+L Device:R R?
+U 1 1 5D545A7F
+P 2850 2500
+AR Path="/5D3E2E6F/5D43B010/5D545A7F" Ref="R?"  Part="1"
+AR Path="/5DB20FE4/5D545A7F" Ref="R?"  Part="1"
+AR Path="/5D3E2E6F/5D43B07B/5D545A7F" Ref="R65"  Part="1"
+F 0 "R65" V 2850 2500 50  0000 C CNN
+F 1 "R 10k" V 2900 2750 50  0000 C CNN
+F 2 "Resistor_SMD:R_1206_3216Metric_Pad1.42x1.75mm_HandSolder" V 2780 2500 50  0001 C CNN
+F 3 "~" H 2850 2500 50  0001 C CNN
+	1    2850 2500
+	0    -1   -1   0
+$EndComp
+Text GLabel 3100 2500 2    50   Input ~ 0
+SH0b
+Wire Wire Line
+	3100 2500 3000 2500
+Wire Wire Line
+	2700 2500 2350 2500
+Wire Wire Line
+	2350 2650 2350 2500
+Connection ~ 2350 2650
+Wire Wire Line
+	2350 2650 2250 2650
 $EndSCHEMATC
