File: Building sensor/Designs/EMI_sensor_control_Rev1.0/file5DAF1840.sch (KiCad schematic (older format))
At the start: 33 parts, among them J1 Conn_01x06_Male, U11 INA163UA_2K5, U12 ADA4096-2ARMZ, U13 INA163UA_2K5

Commit message: Weekly Commit
Weekly Commit 08/09/2019
Parts:
- AE2, AE3: footprint (none) -> Connector_Coaxial:SMA_Custom
- C37, C42: value C -> C 100n; footprint (none) -> Capacitor_SMD:C_1812_4532Metric_Pad1.30x3.40mm_HandSolder
- C38, C41: value C -> C .047u; footprint (none) -> Capacitor_SMD:C_0805_2012Metric_Pad1.15x1.40mm_HandSolder
- J1: footprint (none) -> Connector_PinHeader_2.54mm:PinHeader_1x06_P2.54mm_Vertical
- L3, L4, L5: footprint (none) -> footprints:AISC-1008-1R2G-T
- R33, R34, R41: footprint (none) -> Resistor_SMD:R_1206_3216Metric_Pad1.42x1.75mm_HandSolder
- R35, R47: value R -> R 1.6k; footprint (none) -> Resistor_SMD:R_0805_2012Metric_Pad1.15x1.40mm_HandSolder
- R36, R46: value R -> R 536; footprint (none) -> Resistor_SMD:R_0805_2012Metric_Pad1.15x1.40mm_HandSolder
- R37, R45: footprint (none) -> Resistor_SMD:R_0805_2012Metric_Pad1.15x1.40mm_HandSolder
- R38, R44: value R -> R 3.16k; footprint (none) -> Resistor_SMD:R_0805_2012Metric_Pad1.15x1.40mm_HandSolder
- R39, R43: value R -> R 1.2k; footprint (none) -> Resistor_SMD:R_0805_2012Metric_Pad1.15x1.40mm_HandSolder
- R40, R42: value R -> R 5.36k; footprint (none) -> Resistor_SMD:R_0805_2012Metric_Pad1.15x1.40mm_HandSolder
- U11, U13: footprint (none) -> footprints:INA163UA&slash_2K5
- U12: footprint (none) -> footprints:ADA4096-2ARMZ
Connections:
- net -5V: now also C89.1
Changed lines of the file:
@@
 F 0 "AE2" H 6730 2564 50  0000 L CNN
 F 1 "Antenna_Loop Bx" H 6730 2473 50  0000 L CNN
-F 2 "" H 6500 2550 50  0001 C CNN
+F 2 "Connector_Coaxial:SMA_Custom" H 6500 2550 50  0001 C CNN
 F 3 "~" H 6500 2550 50  0001 C CNN
 	1    6500 2550
@@
 F 0 "AE3" H 7830 2564 50  0000 L CNN
 F 1 "Antenna_Loop Rx" H 7830 2473 50  0000 L CNN
-F 2 "" H 7600 2550 50  0001 C CNN
+F 2 "Connector_Coaxial:SMA_Custom" H 7600 2550 50  0001 C CNN
 F 3 "~" H 7600 2550 50  0001 C CNN
 	1    7600 2550
@@
 F 0 "U11" H 5950 5187 60  0000 C CNN
 F 1 "INA163UA_2K5" H 5950 5081 60  0000 C CNN
-F 2 "" H 5950 5040 60  0001 C CNN
+F 2 "footprints:INA163UA&slash_2K5" H 5950 5040 60  0001 C CNN
 F 3 "" H 4750 4800 60  0000 C CNN
 	1    4750 4800
@@
 F 0 "U13" H 11250 5137 60  0000 C CNN
 F 1 "INA163UA_2K5" H 11250 5031 60  0000 C CNN
-F 2 "" H 11250 4990 60  0001 C CNN
+F 2 "footprints:INA163UA&slash_2K5" H 11250 4990 60  0001 C CNN
 F 3 "" H 10050 4750 60  0000 C CNN
 	1    10050 4750
@@
 F 0 "R37" V 5950 4300 50  0000 C CNN
 F 1 "R 22ohm" V 5834 4300 50  0000 C CNN
-F 2 "" V 5880 4300 50  0001 C CNN
+F 2 "Resistor_SMD:R_0805_2012Metric_Pad1.15x1.40mm_HandSolder" V 5880 4300 50  0001 C CNN
 F 3 "~" H 5950 4300 50  0001 C CNN
 	1    5950 4300
@@
 F 0 "J1" H 9208 3381 50  0000 C CNN
 F 1 "Conn_01x06_Male" H 9208 3290 50  0000 C CNN
-F 2 "" H 9100 3000 50  0001 C CNN
+F 2 "Connector_PinHeader_2.54mm:PinHeader_1x06_P2.54mm_Vertical" H 9100 3000 50  0001 C CNN
 F 3 "~" H 9100 3000 50  0001 C CNN
 	1    9100 3000
@@
 F 0 "R45" V 11250 4250 50  0000 C CNN
 F 1 "R 22ohm" V 11134 4250 50  0000 C CNN
-F 2 "" V 11180 4250 50  0001 C CNN
+F 2 "Resistor_SMD:R_0805_2012Metric_Pad1.15x1.40mm_HandSolder" V 11180 4250 50  0001 C CNN
 F 3 "~" H 11250 4250 50  0001 C CNN
 	1    11250 4250
@@
 BxCoilsig
 Wire Wire Line
-	10050 5250 9800 5250
+	10050 5250 9950 5250
 Wire Wire Line
 	9800 5250 9800 5400
@@
 F 0 "U12" H 8500 7387 60  0000 C CNN
 F 1 "ADA4096-2ARMZ" H 8500 7281 60  0000 C CNN
-F 2 "" H 8500 7240 60  0001 C CNN
+F 2 "footprints:ADA4096-2ARMZ" H 8500 7240 60  0001 C CNN
 F 3 "" H 7300 7000 60  0000 C CNN
 	1    7300 7000
@@
 P 6400 7550
 F 0 "R38" V 6400 7450 50  0000 L CNN
-F 1 "R" H 6470 7505 50  0000 L CNN
-F 2 "" V 6330 7550 50  0001 C CNN
+F 1 "R 3.16k" V 6500 7400 50  0000 L CNN
+F 2 "Resistor_SMD:R_0805_2012Metric_Pad1.15x1.40mm_HandSolder" V 6330 7550 50  0001 C CNN
 F 3 "~" H 6400 7550 50  0001 C CNN
 	1    6400 7550
@@
 P 5200 7600
 F 0 "R36" V 5200 7550 50  0000 L CNN
-F 1 "R" H 5270 7555 50  0000 L CNN
-F 2 "" V 5130 7600 50  0001 C CNN
+F 1 "R 536" H 5270 7555 50  0000 L CNN
+F 2 "Resistor_SMD:R_0805_2012Metric_Pad1.15x1.40mm_HandSolder" V 5130 7600 50  0001 C CNN
 F 3 "~" H 5200 7600 50  0001 C CNN
 	1    5200 7600
@@
 P 4800 7300
 F 0 "R35" V 4800 7300 50  0000 C CNN
-F 1 "R" V 4684 7300 50  0000 C CNN
-F 2 "" V 4730 7300 50  0001 C CNN
+F 1 "R 1.6k" V 4684 7300 50  0000 C CNN
+F 2 "Resistor_SMD:R_0805_2012Metric_Pad1.15x1.40mm_HandSolder" V 4730 7300 50  0001 C CNN
 F 3 "~" H 4800 7300 50  0001 C CNN
 	1    4800 7300
@@
 P 11800 7300
 F 0 "R46" V 11800 7250 50  0000 L CNN
-F 1 "R" H 11870 7255 50  0000 L CNN
-F 2 "" V 11730 7300 50  0001 C CNN
+F 1 "R 536" H 11870 7255 50  0000 L CNN
+F 2 "Resistor_SMD:R_0805_2012Metric_Pad1.15x1.40mm_HandSolder" V 11730 7300 50  0001 C CNN
 F 3 "~" H 11800 7300 50  0001 C CNN
 	1    11800 7300
@@
 P 12200 7600
 F 0 "R47" V 12200 7600 50  0000 C CNN
-F 1 "R" V 12084 7600 50  0000 C CNN
-F 2 "" V 12130 7600 50  0001 C CNN
+F 1 "R 1.6k" V 12084 7600 50  0000 C CNN
+F 2 "Resistor_SMD:R_0805_2012Metric_Pad1.15x1.40mm_HandSolder" V 12130 7600 50  0001 C CNN
 F 3 "~" H 12200 7600 50  0001 C CNN
 	1    12200 7600
@@
 F 0 "R33" V 4100 4800 50  0000 C CNN
 F 1 "R 47" V 3984 4800 50  0000 C CNN
-F 2 "" V 4030 4800 50  0001 C CNN
+F 2 "Resistor_SMD:R_1206_3216Metric_Pad1.42x1.75mm_HandSolder" V 4030 4800 50  0001 C CNN
 F 3 "~" H 4100 4800 50  0001 C CNN
 	1    4100 4800
@@
 F 0 "L3" V 4290 5100 50  0000 C CNN
 F 1 "L 1.2u" V 4199 5100 50  0000 C CNN
-F 2 "" H 4100 5100 50  0001 C CNN
+F 2 "footprints:AISC-1008-1R2G-T" H 4100 5100 50  0001 C CNN
 F 3 "~" H 4100 5100 50  0001 C CNN
 	1    4100 5100
@@
 F 0 "L4" V 4300 5200 50  0000 C CNN
 F 1 "L 1.2u" V 4200 5200 50  0000 C CNN
-F 2 "" H 4100 5200 50  0001 C CNN
+F 2 "footprints:AISC-1008-1R2G-T" H 4100 5200 50  0001 C CNN
 F 3 "~" H 4100 5200 50  0001 C CNN
 	1    4100 5200
@@
 F 0 "R34" V 4100 5500 50  0000 C CNN
 F 1 "R 47" V 4250 5500 50  0000 C CNN
-F 2 "" V 4030 5500 50  0001 C CNN
+F 2 "Resistor_SMD:R_1206_3216Metric_Pad1.42x1.75mm_HandSolder" V 4030 5500 50  0001 C CNN
 F 3 "~" H 4100 5500 50  0001 C CNN
 	1    4100 5500
@@
 F 0 "R41" V 9143 4750 50  0000 C CNN
 F 1 "R 47" V 9234 4750 50  0000 C CNN
-F 2 "" V 9280 4750 50  0001 C CNN
+F 2 "Resistor_SMD:R_1206_3216Metric_Pad1.42x1.75mm_HandSolder" V 9280 4750 50  0001 C CNN
 F 3 "~" H 9350 4750 50  0001 C CNN
 	1    9350 4750
@@
 F 0 "L5" V 9540 5050 50  0000 C CNN
 F 1 "L 1.2u" V 9449 5050 50  0000 C CNN
-F 2 "" H 9350 5050 50  0001 C CNN
+F 2 "footprints:AISC-1008-1R2G-T" H 9350 5050 50  0001 C CNN
 F 3 "~" H 9350 5050 50  0001 C CNN
 	1    9350 5050
@@
 P 5600 7300
 F 0 "C37" V 5371 7300 50  0000 C CNN
-F 1 "C" V 5462 7300 50  0000 C CNN
-F 2 "" H 5600 7300 50  0001 C CNN
+F 1 "C 100n" V 5462 7300 50  0000 C CNN
+F 2 "Capacitor_SMD:C_1812_4532Metric_Pad1.30x3.40mm_HandSolder" H 5600 7300 50  0001 C CNN
 F 3 "~" H 5600 7300 50  0001 C CNN
 	1    5600 7300
@@
 P 6000 7500
 F 0 "C38" H 5908 7454 50  0000 R CNN
-F 1 "C" H 5908 7545 50  0000 R CNN
-F 2 "" H 6000 7500 50  0001 C CNN
+F 1 "C .047u" H 6000 7600 50  0000 R CNN
+F 2 "Capacitor_SMD:C_0805_2012Metric_Pad1.15x1.40mm_HandSolder" H 6000 7500 50  0001 C CNN
 F 3 "~" H 6000 7500 50  0001 C CNN
 	1    6000 7500
@@
 P 6850 7800
 F 0 "R40" V 6850 7800 50  0000 C CNN
-F 1 "R" V 6734 7800 50  0000 C CNN
-F 2 "" V 6780 7800 50  0001 C CNN
+F 1 "R 5.36k" V 6734 7800 50  0000 C CNN
+F 2 "Resistor_SMD:R_0805_2012Metric_Pad1.15x1.40mm_HandSolder" V 6780 7800 50  0001 C CNN
 F 3 "~" H 6850 7800 50  0001 C CNN
 	1    6850 7800
@@
 P 6600 8050
 F 0 "R39" V 6600 8000 50  0000 L CNN
-F 1 "R" H 6670 8005 50  0000 L CNN
-F 2 "" V 6530 8050 50  0001 C CNN
+F 1 "R 1.2k" H 6670 8005 50  0000 L CNN
+F 2 "Resistor_SMD:R_0805_2012Metric_Pad1.15x1.40mm_HandSolder" V 6530 8050 50  0001 C CNN
 F 3 "~" H 6600 8050 50  0001 C CNN
 	1    6600 8050
@@
 P 10600 7350
 F 0 "R44" V 10600 7300 50  0000 L CNN
-F 1 "R" H 10670 7305 50  0000 L CNN
-F 2 "" V 10530 7350 50  0001 C CNN
+F 1 "R 3.16k" V 10700 7250 50  0000 L CNN
+F 2 "Resistor_SMD:R_0805_2012Metric_Pad1.15x1.40mm_HandSolder" V 10530 7350 50  0001 C CNN
 F 3 "~" H 10600 7350 50  0001 C CNN
 	1    10600 7350
@@
 P 11000 7400
 F 0 "C41" H 10908 7354 50  0000 R CNN
-F 1 "C" H 10908 7445 50  0000 R CNN
-F 2 "" H 11000 7400 50  0001 C CNN
+F 1 "C .047u" H 11000 7500 50  0000 R CNN
+F 2 "Capacitor_SMD:C_0805_2012Metric_Pad1.15x1.40mm_HandSolder" H 11000 7400 50  0001 C CNN
 F 3 "~" H 11000 7400 50  0001 C CNN
 	1    11000 7400
@@
 P 10400 6850
 F 0 "R43" V 10400 6800 50  0000 L CNN
-F 1 "R" H 10470 6805 50  0000 L CNN
-F 2 "" V 10330 6850 50  0001 C CNN
+F 1 "R 1.2k" H 10470 6805 50  0000 L CNN
+F 2 "Resistor_SMD:R_0805_2012Metric_Pad1.15x1.40mm_HandSolder" V 10330 6850 50  0001 C CNN
 F 3 "~" H 10400 6850 50  0001 C CNN
 	1    10400 6850
@@
 P 11400 7600
 F 0 "C42" V 11171 7600 50  0000 C CNN
-F 1 "C" V 11262 7600 50  0000 C CNN
-F 2 "" H 11400 7600 50  0001 C CNN
+F 1 "C 100n" V 11262 7600 50  0000 C CNN
+F 2 "Capacitor_SMD:C_1812_4532Metric_Pad1.30x3.40mm_HandSolder" H 11400 7600 50  0001 C CNN
 F 3 "~" H 11400 7600 50  0001 C CNN
 	1    11400 7600
@@
 P 10150 7100
 F 0 "R42" V 10150 7100 50  0000 C CNN
-F 1 "R" V 10034 7100 50  0000 C CNN
-F 2 "" V 10080 7100 50  0001 C CNN
+F 1 "R 5.36k" V 10034 7100 50  0000 C CNN
+F 2 "Resistor_SMD:R_0805_2012Metric_Pad1.15x1.40mm_HandSolder" V 10080 7100 50  0001 C CNN
 F 3 "~" H 10150 7100 50  0001 C CNN
 	1    10150 7100
@@
 $EndComp
 Wire Wire Line
-	9950 5250 9950 5350
-Wire Wire Line
 	9950 5550 9950 5650
+Wire Wire Line
+	9950 5350 9950 5250
+Connection ~ 9950 5250
+Wire Wire Line
+	9950 5250 9800 5250
 $EndSCHEMATC

Commit message: End of Rev 1.01
End of Rev 1.01 change will be made to Rx and Bx connection in 1.02
Parts:
- AE2, AE3: footprint Connector_Coaxial:SMA_Custom -> Connector_Coaxial:SMA_Molex_73251-2200_Horizontal
Changed lines of the file:
@@
 F 0 "AE2" H 6730 2564 50  0000 L CNN
 F 1 "Antenna_Loop Bx" H 6730 2473 50  0000 L CNN
-F 2 "Connector_Coaxial:SMA_Custom" H 6500 2550 50  0001 C CNN
+F 2 "Connector_Coaxial:SMA_Molex_73251-2200_Horizontal" H 6500 2550 50  0001 C CNN
 F 3 "~" H 6500 2550 50  0001 C CNN
 	1    6500 2550
@@
 F 0 "AE3" H 7830 2564 50  0000 L CNN
 F 1 "Antenna_Loop Rx" H 7830 2473 50  0000 L CNN
-F 2 "Connector_Coaxial:SMA_Custom" H 7600 2550 50  0001 C CNN
+F 2 "Connector_Coaxial:SMA_Molex_73251-2200_Horizontal" H 7600 2550 50  0001 C CNN
 F 3 "~" H 7600 2550 50  0001 C CNN
 	1    7600 2550

Commit message: weekly commit
weekly commit, First of Rev 1.02
Parts:
- removed J1: Conn_01x06_Male, Connector_PinHeader_2.54mm:PinHeader_1x06_P2.54mm_Vertical, symbol Connector:Conn_01x06_Male
Connections:
- net BxOut is gone; now on net GND: AE2.2
- net BxCoilsig: now also AE3.2, L3.1, R33.2
- net GND: no longer AE3.2
- net RxCoilsig+: now also AE3.1
- removed net RxCoilsig-: AE3.1, L3.1, R33.2
Other:
- moved on the sheet: AE2
Changed lines of the file:
@@
 Title "Pancreas EMI Conductivity Meter "
 Date ""
-Rev ""
+Rev "1.02"
 Comp ""
 Comment1 ""
@@
 F 3 "~" H 6500 2550 50  0001 C CNN
 	1    6500 2550
-	1    0    0    -1
+	-1   0    0    -1
 $EndComp
 $Comp
 L Device:Antenna_Loop AE3
 U 1 1 5DAFD1FF
-P 7600 2550
-F 0 "AE3" H 7830 2564 50  0000 L CNN
-F 1 "Antenna_Loop Rx" H 7830 2473 50  0000 L CNN
-F 2 "Connector_Coaxial:SMA_Molex_73251-2200_Horizontal" H 7600 2550 50  0001 C CNN
-F 3 "~" H 7600 2550 50  0001 C CNN
-	1    7600 2550
-	1    0    0    -1
-$EndComp
-Wire Wire Line
-	7600 2750 7600 3150
-Wire Wire Line
-	6600 3150 6600 2750
+P 7700 2550
+F 0 "AE3" H 7930 2564 50  0000 L CNN
+F 1 "Antenna_Loop Rx" H 7930 2473 50  0000 L CNN
+F 2 "Connector_Coaxial:SMA_Molex_73251-2200_Horizontal" H 7700 2550 50  0001 C CNN
+F 3 "~" H 7700 2550 50  0001 C CNN
+	1    7700 2550
+	-1   0    0    -1
+$EndComp
 $Comp
 L power:GND #PWR082
 U 1 1 5DAFD207
-P 7700 3150
-F 0 "#PWR082" H 7700 2900 50  0001 C CNN
-F 1 "GND" H 7750 3000 50  0000 C CNN
-F 2 "" H 7700 3150 50  0001 C CNN
-F 3 "" H 7700 3150 50  0001 C CNN
-	1    7700 3150
+P 6400 3150
+F 0 "#PWR082" H 6400 2900 50  0001 C CNN
+F 1 "GND" H 6450 3000 50  0000 C CNN
+F 2 "" H 6400 3150 50  0001 C CNN
+F 3 "" H 6400 3150 50  0001 C CNN
+	1    6400 3150
 	1    0    0    -1
 $EndComp
@@
 Wire Wire Line
 	7300 4300 6100 4300
-Text GLabel 9600 2550 2    50   Input ~ 0
+Text GLabel 7100 3200 3    50   Input ~ 0
 RxCoilsig-
-Text GLabel 6500 3150 3    50   Input ~ 0
+Text GLabel 6900 3200 3    50   Input ~ 0
 BxCoilsig
-$Comp
-L power:GND #PWR086
-U 1 1 5DAFD229
-P 9600 3150
-F 0 "#PWR086" H 9600 2900 50  0001 C CNN
-F 1 "GND" H 9605 2977 50  0000 C CNN
-F 2 "" H 9600 3150 50  0001 C CNN
-F 3 "" H 9600 3150 50  0001 C CNN
-	1    9600 3150
-	0    -1   -1   0
-$EndComp
-Text GLabel 9600 2700 2    50   Input ~ 0
-RxOut
-Text GLabel 6600 3150 3    50   Input ~ 0
-BxOut
-Text GLabel 7600 3150 3    50   Input ~ 0
-RxOut
 Wire Wire Line
 	7700 3150 7700 2750
-Wire Wire Line
-	6500 2750 6500 3150
-Wire Wire Line
-	9300 3000 9600 3000
-Wire Wire Line
-	9300 2900 9400 2900
-Wire Wire Line
-	9400 2900 9400 2850
-Wire Wire Line
-	9400 2850 9600 2850
-Wire Wire Line
-	9300 2800 9450 2800
-Wire Wire Line
-	9450 2800 9450 2700
-Wire Wire Line
-	9450 2700 9600 2700
-Wire Wire Line
-	9450 2700 9450 2550
-Wire Wire Line
-	9450 2550 9600 2550
-Connection ~ 9450 2700
 Text GLabel 3700 5100 0    50   Input ~ 0
 RxCoilsig-
@@
 Text GLabel 3700 5200 0    50   Input ~ 0
 RxCoilsig+
-Text GLabel 9600 3300 2    50   Input ~ 0
+Text GLabel 7700 3150 3    50   Input ~ 0
 RxCoilsig+
-Text GLabel 9600 3450 2    50   Input ~ 0
-BxCoilsig
-$Comp
-L power:GND #PWR085
-U 1 1 5DAFD252
-P 9600 3000
-F 0 "#PWR085" H 9600 2750 50  0001 C CNN
-F 1 "GND" H 9605 2827 50  0000 C CNN
-F 2 "" H 9600 3000 50  0001 C CNN
-F 3 "" H 9600 3000 50  0001 C CNN
-	1    9600 3000
-	0    -1   -1   0
-$EndComp
-Text GLabel 9600 2850 2    50   Input ~ 0
-BxOut
-$Comp
-L Connector:Conn_01x06_Male J1
-U 1 1 5DAFD259
-P 9100 3000
-F 0 "J1" H 9208 3381 50  0000 C CNN
-F 1 "Conn_01x06_Male" H 9208 3290 50  0000 C CNN
-F 2 "Connector_PinHeader_2.54mm:PinHeader_1x06_P2.54mm_Vertical" H 9100 3000 50  0001 C CNN
-F 3 "~" H 9100 3000 50  0001 C CNN
-	1    9100 3000
-	1    0    0    -1
-$EndComp
-Wire Wire Line
-	9300 3100 9450 3100
-Wire Wire Line
-	9450 3100 9450 3150
-Wire Wire Line
-	9450 3150 9600 3150
-Wire Wire Line
-	9300 3200 9400 3200
-Wire Wire Line
-	9400 3200 9400 3300
-Wire Wire Line
-	9400 3300 9600 3300
-Wire Wire Line
-	9300 3300 9350 3300
-Wire Wire Line
-	9350 3300 9350 3450
-Wire Wire Line
-	9350 3450 9600 3450
 Text GLabel 12700 5550 3    50   Input ~ 0
 BxCoilAmp
@@
 Wire Wire Line
 	9950 5250 9800 5250
+Wire Wire Line
+	6900 3200 6900 2950
+Wire Wire Line
+	6900 2950 7100 2950
+Wire Wire Line
+	7100 3200 7100 2950
+Connection ~ 7100 2950
+Wire Wire Line
+	7100 2950 7600 2950
+Wire Wire Line
+	6500 2750 6500 2950
+Wire Wire Line
+	6900 2950 6500 2950
+Connection ~ 6900 2950
+Wire Wire Line
+	6400 2750 6400 3150
+Wire Wire Line
+	7600 2750 7600 2950
 $EndSCHEMATC
