File: Building sensor/Designs/EMI_sensor_control_Rev2.0/file5D278C8E.sch (KiCad schematic (older format))
At the start: 12 parts, among them Q1 BSR14, Q2 BSR14, Q3 DMHC3025LSD-13

Commit message: backup
2/04/2020
Parts:
- added C?: C, symbol Device:C
- added C?: C 10u, symbol Device:C
- added C? (x6): C .1u, symbol Device:C
- added C?: C 1n, symbol Device:C
- added C?: C 1u, symbol Device:C
- added D?: B140-E3, Diode_SMD:D_SMA, symbol Diode:B140-E3
- added L?: L 5.5u, symbol Device:L
- added Q?: CMST3904_TR_CMST3904_TR, SOT65P210X110-3N, symbol FinalProject-cache:CMST3904_TR_CMST3904_TR
- added Q?: MMBT3906, Package_TO_SOT_SMD:SOT-23, symbol Transistor_BJT:MMBT3906
- added R? (x4): R, symbol Device:R
- added R?: R 5.1k, symbol Device:R
- added R?: R 60.4k, symbol Device:R
- added R?: R 1k, symbol Device:R
- added R?: R 4.99k, symbol Device:R
- added R? (x2): R 100k, symbol Device:R
- added TP?: TestPoint, symbol Connector:TestPoint
- added U?: LT3092EST_PBF, digikey-footprints:TO-261-4, symbol dk_PMIC-Current-Regulation-Management:LT3092EST_PBF
- added U?: SI2309CDS-T1-GE3, TO-236, symbol FinalProject-cache:2019-12-05_20-48-20_SI2309CDS-T1-GE3
- added U?: LT8610, Package_SO:LTC_MSOP-16-1EP_3x4mm_P0.5mm_EP2.15x3.26mm, symbol Regulator_Switching:LT8610
- added U?: 2019-12-05_20-39-13_LT3081EFE-PBF, TSSOP-16_FE/BB, symbol FinalProject-cache:2019-12-05_20-39-13_LT3081EFE-PBF
Connections:
- net +BATT: now also C?.1, R?.1, U?.3 (D), U?.5 (VIN), U?.6 (VIN); no longer Q3.7 (P1S/P2S), R4.1
- net GND: now also C?.1, C?.1, C?.1, C?.1, C?.2, C?.2, C?.2, C?.2, R?.1, R?.1, R?.1, U?.17 (GND), U?.7 (GND), U?.8 (GND)
- new net: R?.2, U?.1 (SET)
- new net: R?.1, U?.2 (OUT), U?.4 (TAB/OUT)
- new net: C?.1, U?.2 (S), U?.3 (IN)
- new net: Q?.2, R?.2
- new net: Q?.3, R?.2, U?.1 (G)
- new net: C?.1, L?.2, U?.10 (SW), U?.11 (SW), U?.9 (SW)
- new net: C?.2, U?.12 (BST)
- new net: R?.1, U?.15 (PG)
- new net: C?.2, Q?.3 (C), R?.2, U?.16 (FB)
- new net: C?.1, U?.2 (TR/SS)
- new net: R?.2, U?.3 (RT)
- new net: Q?.1 (B), R?.1, R?.2
- new net: Q?.2 (E), R?.1
- new net: D?.2 (A), R?.1, R?.2, U?.7 (SET)
- new net: C?.1, R?.2
- new net 3081IN: C?.2, C?.2, C?.2, C?.2, L?.1, R?.2, R?.2, TP?.1, U?.14 (BIAS)
- new net INTVcc: C?.1, Q?.1, U?.1 (SYNC), U?.13 (INTVcc)
- new net Vvar: D?.1 (K), Q3.7 (P1S/P2S), R4.1, R?.1
Other:
- moved on the sheet: AE1, Q1, Q2, Q3, R1, R2, R3, R4, R5, R6, R7, R8

Commit message: Back up
Backup of rev 2.0 for board
Parts:
- removed Q1, Q2: BSR14, Package_TO_SOT_SMD:SOT-23_Handsoldering, symbol Transistor_BJT:BSR14
- removed Q3: DMHC3025LSD-13, digikey-footprints:SOIC-8_W3.9mm, symbol EMI_sensor_control_Rev2.0-rescue:DMHC3025LSD-13-dk_Transistors-FETs-MOSFETs-Arr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
- removed R1, R2, R3, R5, R7, R8: R 1k, Resistor_SMD:R_0805_2012Metric_Pad1.15x1.40mm_HandSolder, symbol Device:R
- removed R4, R6: R 4.7k, Resistor_SMD:R_0805_2012Metric_Pad1.15x1.40mm_HandSolder, symbol Device:R
- removed R?: R, symbol Device:R
- added C? (x9): C .1u, symbol Device:C
- added C?: C 330u, symbol Device:C
- added C? (x5): C 1u, symbol Device:C
- added C?: C 47u, symbol Device:C
- added C?: C 1000u, symbol Device:C
- added C?: C 10n, symbol Device:C
- added C?: C 2700p, symbol Device:C
- added L? (x4): L 50n, symbol Device:L
- added R?: 3386P-1-503LF, POT_3386P, symbol 2020-02-06_16-05-16:3386P-1-503LF
- added R?: R 3.3k, symbol Device:R
- added R? (x2): R 10k, symbol Device:R
- added R?: R 150k, Resistor_SMD:R_0805_2012Metric_Pad1.15x1.40mm_HandSolder, symbol Device:R
- added R?: R 1, Resistor_SMD:R_0805_2012Metric_Pad1.15x1.40mm_HandSolder, symbol Device:R
- added R?: R 3.3, Resistor_SMD:R_0805_2012Metric_Pad1.15x1.40mm_HandSolder, symbol Device:R
- added R?: R 590, Resistor_SMD:R_0805_2012Metric_Pad1.15x1.40mm_HandSolder, symbol Device:R
- added TP? (x2): TestPoint, symbol Connector:TestPoint
- added U?: MCP41HV51-103E_ST, TSSOP14_MC, symbol 2020-02-06_20-31-41:MCP41HV51-103E_ST
- added U?: DRV8412DDWR, DDW44_8P26X4P31, symbol 2020-02-25_19-55-49:DRV8412DDWR
- R?: value R -> R 200
Connections:
- net +BATT: now also C?.1, C?.1, C?.1, C?.2, C?.2, C?.2, C?.2, U?.1 (GVDD_C), U?.14 (V+), U?.2 (VDD), U?.22 (GVDD_B), U?.23 (GVDD_B), U?.44 (GVDD_D)
- net 3081IN: now also C?.1, R?.2, U?.12 (IN), U?.13 (IN), U?.14 (IN), U?.15 (IN)
- net GND: now also C?.1, C?.1, C?.1, C?.1, C?.1, C?.1, C?.1, C?.1, C?.1, C?.1, C?.2, C?.2, C?.2, R?.2, R?.2, U?.10 (V-), U?.13 (GND), U?.13 (P0A), U?.19 (NC), U?.20 (NC), U?.25 (NC), U?.29 (GND_A), U?.3 (NC), U?.30 (GND_B), U?.37 (GND_C), U?.38 (GND_D), U?.4 (NC), U?.42 (NC), U?.5 (PWM_D), U?.6 (*WLAT), U?.7 (PWM_C), U?.8 (NC), U?.9 (DGND), U?.EPAD
- net TxC1: now also U?.17 (PWM_A)
- net TxC2: now also U?.15 (PWM_B)
- net Vvar: now also U?.1 (OUT), U?.11 (TEMP), U?.16 (OUT), U?.17 (OUT), U?.2 (OUT), U?.3 (OUT), U?.4 (OUT), U?.5 (OUT), U?.8 (OUT), U?.9 (OUT), C?.2, C?.2, C?.2, C?.2, C?.2, R?.2, R?.2, U?.26 (PVDD_A), U?.27 (PVDD_A), U?.32 (PVDD_B), U?.35 (PVDD_C), U?.40 (PVDD_D), U?.41 (PVDD_D)
- net at AE1.1: now also C?.2, R?.1, TP?.1
- net at AE1.2: now also C?.1, L?.1, L?.1, TP?.1
- net at U?.1 (SET): now also R?.3
- net IMon: now reaches U?.10 (IMON)
- net IMon: now also R?.1
- net at U?.6 (ILIM): now also R?.1
- net at D?.2 (A), R?.2, U?.7 (SET): now also R?.2, U?.11 (P0B), U?.12 (P0W)
- new net: R?.1, U?.7 (*SHDN)
- new net: C?.1, R?.1, R?.2, U?.10 (M3), U?.12 (AGND), U?.8 (M1)
- new net: C?.2, U?.11 (VREG), U?.9 (M2)
- new net: R?.1, U?.14 (OC_ADJ)
- new net: C?.2, U?.24 (BST_A)
- new net: C?.1, L?.2, U?.28 (OUT_A)
- new net: C?.1, L?.2, U?.31 (OUT_B)
- new net: C?.2, U?.33 (BST_B)
- new net: C?.2, U?.34 (BST_C)
- new net: C?.1, L?.2, U?.36 (OUT_C)
- new net: C?.1, L?.2, U?.39 (OUT_D)
- new net: C?.2, U?.43 (BST_D)
- new net: L?.1, L?.1, R?.2
- new net: C?.2, R?.1
- new net +3V3: R?.2, U?.1 (VL)
- new net RCS: U?.3 (*CS)
- new net RMISO: U?.5 (SDO)
- new net RMOSI: U?.4 (SDI)
- new net RSCK: U?.2 (SCK)
- new net RSET_AD: U?.18 (*FAULT)
- new net RSET_CD: U?.6 (*RESET_CD)
- no-connect marks 0 -> 1
Other:
- moved on the sheet: AE1, C?, D?, L?, Q?, R?, TP?, U?

Commit message: Rev 2.0 Complete
Rev 2.0 of PCB Completed
SCHM, PCB layout, and gerber files generated
Parts:
- C1, C17, C2, C28, C3, C4, C5: renamed from C?; footprint (none) -> Capacitor_SMD:C_0805_2012Metric_Pad1.15x1.40mm_HandSolder
- C10, C11, C12, C14, C18, C19, C20, C22, C24, C25, C26, C27, C7, C8, C9: renamed from C?; value C .1u -> C 100n; footprint (none) -> Capacitor_SMD:C_0603_1608Metric_Pad1.05x0.95mm_HandSolder
- C13, C21: renamed from C?; footprint (none) -> Capacitor_SMD:C_0603_1608Metric_Pad1.05x0.95mm_HandSolder
- C15: renamed from C?; footprint (none) -> Capacitor_SMD:CP_Elec_10x10
- C16: renamed from C?; footprint (none) -> Capacitor_SMD:C_1206_3216Metric_Pad1.42x1.75mm_HandSolder
- C23: renamed from C?; value C 1000u -> C 470u; footprint (none) -> Capacitor_SMD:CP_Elec_10x10
- C29: renamed from C?; value C -> C 1u; footprint (none) -> Capacitor_SMD:C_0805_2012Metric_Pad1.15x1.40mm_HandSolder
- C6: renamed from C?; footprint (none) -> Capacitor_SMD:C_1210_3225Metric_Pad1.42x2.65mm_HandSolder
- L1: renamed from L?; footprint (none) -> Inductor_SMD:L_Wuerth_HCI-1050
- L2, L3, L4, L5: renamed from L?; value L 50n -> L 51n; footprint (none) -> Inductor_SMD:L_0805_2012Metric_Pad1.15x1.40mm_HandSolder
- Q2: renamed from Q?; footprint SOT65P210X110-3N -> Package_TO_SOT_SMD:SOT-323_SC-70_Handsoldering
- R1, R11, R12, R13, R15, R2, R3, R4, R5, R8: renamed from R?; footprint (none) -> Resistor_SMD:R_0805_2012Metric_Pad1.15x1.40mm_HandSolder
- R14: renamed from R?; footprint POT_3386P -> Potentiometer_THT:Potentiometer_Bourns_3386P_Vertical
- R16: renamed from R?; value R -> R 5.1k; footprint (none) -> Resistor_SMD:R_0805_2012Metric_Pad1.15x1.40mm_HandSolder
- R17: renamed from R?; value R -> R 2.7k; footprint (none) -> Resistor_SMD:R_0805_2012Metric_Pad1.15x1.40mm_HandSolder
- R6: renamed from R?; value R 590 -> R 590; footprint Resistor_SMD:R_0805_2012Metric_Pad1.15x1.40mm_HandSolder -> Resistor_SMD:R_1206_3216Metric_Pad1.42x1.75mm_HandSolder
- TP1, TP2, TP3: renamed from TP?; footprint (none) -> TestPoint:TestPoint_Pad_D3.0mm
- U1: renamed from U?; footprint Package_SO:LTC_MSOP-16-1EP_3x4mm_P0.5mm_EP2.15x3.26mm -> Package_SO:MSOP-16-1EP_3x4mm_P0.5mm_EP1.65x2.85mm_ThermalVias
- U2: renamed from U?; footprint DDW44_8P26X4P31 -> Package_SO:SOIC-44
- U3: renamed from U?; footprint TSSOP-16_FE/BB -> Package_SO:TSSOP-16-1EP_4.4x5mm_P0.65mm; symbol FinalProject-cache:2019-12-05_20-39-13_LT3081EFE-PBF -> EMI_sensor_control_Rev2.0-rescue:2019-12-05_20-39-13_LT3081EFE-PBF-FinalProject-cache
- U4: renamed from U?; footprint TSSOP14_MC -> Package_SO:TSSOP-14_4.4x5mm_P0.65mm
- U6: renamed from U?; footprint TO-236 -> Package_TO_SOT_SMD:SOT-23; symbol FinalProject-cache:2019-12-05_20-48-20_SI2309CDS-T1-GE3 -> EMI_sensor_control_Rev2.0-rescue:2019-12-05_20-48-20_SI2309CDS-T1-GE3-FinalProject-cache
- gave numbers to parts that had none: 6
Connections:
- net Pwr1: now reaches U1.4 (EN/UV)
- net RSET_AB: now reaches U2.16 (*RESET_AB)
- net Tx_OTW: now reaches U2.21 (*OTW)
- net RCS renamed Tx_CS
- net RMISO renamed Tx_MISO
- net RMOSI renamed Tx_MOSI
- net RSCK renamed Tx_CLK
- net RSET_AD renamed Tx_Fault
Other:
- moved on the sheet: R15
