File: Building sensor/Designs/EMI_sensor_control_Rev2.0/file5D27CADE.sch (KiCad schematic (older format))
At the start: 46 parts, among them J4 PJ-002AH-SMT-TR, SW1 SW_SP3T, U1 LMZM23601, U2 LMZM23601V5, U3 LMZM23601, U4 LMZM23601, U5 REF2041AIDDCT, U6 LMR23610ADDAR, U7 ADG419BR

Commit message: overdue backup
Parts:
- D4: value LED -> LED Power
- D5: value LED -> LED On
- R66, R67: value R 100 -> R 10k
Connections:
- net +BATT: now also R66.1
- net GND: now also D4.1 (K), D5.1 (K); no longer R66.2, R67.2
- net Pwr1: now also R67.1; no longer D4.2 (A)
- net at D2.A, U7.1: no longer D5.2 (A)
- new net: D5.2 (A), R67.2
- new net: D4.2 (A), R66.2
Other:
- moved on the sheet: D4, D5, R66, R67
Changed lines of the file:
@@
 $Descr A3 16535 11693
 encoding utf-8
-Sheet 3 9
+Sheet 3 8
 Title "Pancreas EMI Conductivity Meter "
 Date ""
@@
 Wire Wire Line
 	13000 8600 13000 8750
-Wire Wire Line
-	12250 8500 12100 8500
 Text GLabel 11350 8500 0    50   Input ~ 0
 Pwr1
-Wire Wire Line
-	11600 8500 11500 8500
 Wire Wire Line
 	13750 8400 13600 8400
@@
 L Device:LED D5
 U 1 1 5D88B2A6
-P 12100 8750
-F 0 "D5" V 12139 8633 50  0000 R CNN
-F 1 "LED" V 12048 8633 50  0000 R CNN
-F 2 "LED_SMD:LED_1206_3216Metric_Pad1.42x1.75mm_HandSolder" H 12100 8750 50  0001 C CNN
-F 3 "~" H 12100 8750 50  0001 C CNN
-	1    12100 8750
+P 8150 8200
+F 0 "D5" V 8189 8083 50  0000 R CNN
+F 1 "LED On" V 8098 8083 50  0000 R CNN
+F 2 "LED_SMD:LED_1206_3216Metric_Pad1.42x1.75mm_HandSolder" H 8150 8200 50  0001 C CNN
+F 3 "~" H 8150 8200 50  0001 C CNN
+	1    8150 8200
 	0    -1   -1   0
 $EndComp
@@
 L power:GND #PWR085
 U 1 1 5D88C49E
-P 12100 9500
-F 0 "#PWR085" H 12100 9250 50  0001 C CNN
-F 1 "GND" H 12105 9327 50  0000 C CNN
-F 2 "" H 12100 9500 50  0001 C CNN
-F 3 "" H 12100 9500 50  0001 C CNN
-	1    12100 9500
-	1    0    0    -1
-$EndComp
-Wire Wire Line
-	12100 8500 12100 8600
-Connection ~ 12100 8500
-Wire Wire Line
-	12100 8500 12000 8500
-Wire Wire Line
-	12100 9350 12100 9500
+P 8150 8500
+F 0 "#PWR085" H 8150 8250 50  0001 C CNN
+F 1 "GND" H 8155 8327 50  0000 C CNN
+F 2 "" H 8150 8500 50  0001 C CNN
+F 3 "" H 8150 8500 50  0001 C CNN
+	1    8150 8500
+	1    0    0    -1
+$EndComp
+Wire Wire Line
+	8150 7950 8150 8050
+Wire Wire Line
+	8150 8350 8150 8500
 $Comp
 L Device:LED D4
 U 1 1 5D8AAF83
-P 11500 8750
-F 0 "D4" V 11539 8633 50  0000 R CNN
-F 1 "LED" V 11448 8633 50  0000 R CNN
-F 2 "LED_SMD:LED_1206_3216Metric_Pad1.42x1.75mm_HandSolder" H 11500 8750 50  0001 C CNN
-F 3 "~" H 11500 8750 50  0001 C CNN
-	1    11500 8750
+P 8650 8200
+F 0 "D4" V 8689 8083 50  0000 R CNN
+F 1 "LED Power" V 8598 8083 50  0000 R CNN
+F 2 "LED_SMD:LED_1206_3216Metric_Pad1.42x1.75mm_HandSolder" H 8650 8200 50  0001 C CNN
+F 3 "~" H 8650 8200 50  0001 C CNN
+	1    8650 8200
 	0    -1   -1   0
 $EndComp
@@
 L power:GND #PWR076
 U 1 1 5D8AAF8F
-P 11500 9500
-F 0 "#PWR076" H 11500 9250 50  0001 C CNN
-F 1 "GND" H 11505 9327 50  0000 C CNN
-F 2 "" H 11500 9500 50  0001 C CNN
-F 3 "" H 11500 9500 50  0001 C CNN
-	1    11500 9500
-	1    0    0    -1
-$EndComp
-Wire Wire Line
-	11500 9350 11500 9500
-Wire Wire Line
-	11500 8600 11500 8500
-Connection ~ 11500 8500
-Wire Wire Line
-	11500 8500 11350 8500
-Wire Wire Line
-	11500 8900 11500 9050
+P 8650 8500
+F 0 "#PWR076" H 8650 8250 50  0001 C CNN
+F 1 "GND" H 8655 8327 50  0000 C CNN
+F 2 "" H 8650 8500 50  0001 C CNN
+F 3 "" H 8650 8500 50  0001 C CNN
+	1    8650 8500
+	1    0    0    -1
+$EndComp
+Wire Wire Line
+	8650 8350 8650 8500
+Wire Wire Line
+	8650 8050 8650 7950
+Wire Wire Line
+	8650 7500 8650 7650
 $Comp
 L Device:R R?
 U 1 1 5D8D36A1
-P 11500 9200
+P 8650 7800
 AR Path="/5D8D36A1" Ref="R?"  Part="1"
 AR Path="/5D2792E3/5D8D36A1" Ref="R?"  Part="1"
 AR Path="/5D27CADF/5D8D36A1" Ref="R66"  Part="1"
-F 0 "R66" H 11570 9246 50  0000 L CNN
-F 1 "R 100" H 11570 9155 50  0000 L CNN
-F 2 "Resistor_SMD:R_1206_3216Metric_Pad1.42x1.75mm_HandSolder" V 11430 9200 50  0001 C CNN
-F 3 "~" H 11500 9200 50  0001 C CNN
-	1    11500 9200
-	1    0    0    -1
-$EndComp
-Wire Wire Line
-	12100 8900 12100 9050
+F 0 "R66" H 8720 7846 50  0000 L CNN
+F 1 "R 10k" H 8720 7755 50  0000 L CNN
+F 2 "Resistor_SMD:R_1206_3216Metric_Pad1.42x1.75mm_HandSolder" V 8580 7800 50  0001 C CNN
+F 3 "~" H 8650 7800 50  0001 C CNN
+	1    8650 7800
+	1    0    0    -1
+$EndComp
+Wire Wire Line
+	8150 7500 8150 7650
 $Comp
 L Device:R R?
 U 1 1 5D8DD9FA
-P 12100 9200
+P 8150 7800
 AR Path="/5D8DD9FA" Ref="R?"  Part="1"
 AR Path="/5D2792E3/5D8DD9FA" Ref="R?"  Part="1"
 AR Path="/5D27CADF/5D8DD9FA" Ref="R67"  Part="1"
-F 0 "R67" H 12170 9246 50  0000 L CNN
-F 1 "R 100" H 12170 9155 50  0000 L CNN
-F 2 "Resistor_SMD:R_1206_3216Metric_Pad1.42x1.75mm_HandSolder" V 12030 9200 50  0001 C CNN
-F 3 "~" H 12100 9200 50  0001 C CNN
-	1    12100 9200
-	1    0    0    -1
-$EndComp
+F 0 "R67" H 8220 7846 50  0000 L CNN
+F 1 "R 10k" H 8220 7755 50  0000 L CNN
+F 2 "Resistor_SMD:R_1206_3216Metric_Pad1.42x1.75mm_HandSolder" V 8080 7800 50  0001 C CNN
+F 3 "~" H 8150 7800 50  0001 C CNN
+	1    8150 7800
+	1    0    0    -1
+$EndComp
+Wire Wire Line
+	12000 8500 12250 8500
+Wire Wire Line
+	11350 8500 11600 8500
+Text GLabel 8150 7500 1    50   Input ~ 0
+Pwr1
+$Comp
+L power:+BATT #PWR?
+U 1 1 5DF2B45E
+P 8650 7500
+F 0 "#PWR?" H 8650 7350 50  0001 C CNN
+F 1 "+BATT" H 8665 7673 50  0000 C CNN
+F 2 "" H 8650 7500 50  0001 C CNN
+F 3 "" H 8650 7500 50  0001 C CNN
+	1    8650 7500
+	1    0    0    -1
+$EndComp

Commit message: Back up
Backup of rev 2.0 for board
Parts:
- removed C10: C 10u, Capacitor_SMD:C_1210_3225Metric_Pad1.42x2.65mm_HandSolder, symbol Device:C
- removed C12: C 2.2u, Capacitor_SMD:C_0603_1608Metric_Pad1.05x0.95mm_HandSolder, symbol Device:C
- removed C14: C 100n, Capacitor_SMD:C_0603_1608Metric_Pad1.05x0.95mm_HandSolder, symbol Device:C
- removed C16: C 330u, Capacitor_SMD:CP_Elec_5x5.3, symbol Device:C
- removed C87: C 1.8n, Capacitor_SMD:C_0805_2012Metric_Pad1.15x1.40mm_HandSolder, symbol Device:C
- removed L1: L 6.8u, footprints:SRN6045-6R8Y, symbol Device:L
- removed R15: R 4.42k, Resistor_SMD:R_1206_3216Metric_Pad1.42x1.75mm_HandSolder, symbol Device:R
- removed R16: R 22.1k, Resistor_SMD:R_1206_3216Metric_Pad1.42x1.75mm_HandSolder, symbol Device:R
- removed U6: LMR23610ADDAR, footprints:LMR23610ADDAR, symbol 2019-07-25_16-42-24:LMR23610ADDAR
- R13: value R 38.3k -> R
- R14: value R 25.5k -> R
Connections:
- net +2V5 renamed +3V0
Other:
- moved on the sheet: C11, C13, C15, U5

Commit message: Rev 2.0 Complete
Rev 2.0 of PCB Completed
SCHM, PCB layout, and gerber files generated
Parts:
- removed C11, C13, C15: C 100n, Capacitor_SMD:C_0603_1608Metric_Pad1.05x0.95mm_HandSolder, symbol Device:C
- removed D2: B340A-13-F, digikey-footprints:DO-214AC, symbol dk_Diodes-Rectifiers-Single:B340A-13-F
- removed SW1: SW_SP3T, Button_Switch_SMD:SW_SP3T_PCM13, symbol Switch:SW_SP3T
- removed U5: REF2041AIDDCT, footprints:REF2041AIDDCT, symbol 2019-07-29_16-20-46:REF2041AIDDCT
- removed U7: ADG419BR, Package_SO:SOIC-8_3.9x4.9mm_P1.27mm, symbol Analog_Switch:ADG419BR
- added C32: C 1u, Capacitor_SMD:C_1206_3216Metric_Pad1.42x1.75mm_HandSolder, symbol Device:C_Small
- added C33: C 22u, Capacitor_SMD:C_1206_3216Metric_Pad1.42x1.75mm_HandSolder, symbol Device:C_Small
- added C34: C 1u, Capacitor_SMD:C_0805_2012Metric_Pad1.15x1.40mm_HandSolder, symbol Device:C_Small
- added C36, C40: C 100n, Capacitor_SMD:C_0603_1608Metric_Pad1.05x0.95mm_HandSolder, symbol Device:C_Small
- added C37, C38, C41, C42: C 10u, Capacitor_SMD:C_1210_3225Metric_Pad1.42x2.65mm_HandSolder, symbol Device:C_Small
- added R20: R 102k, Resistor_SMD:R_0805_2012Metric_Pad1.15x1.40mm_HandSolder, symbol Device:R
- added R21: R 25.5k, Resistor_SMD:R_0805_2012Metric_Pad1.15x1.40mm_HandSolder, symbol Device:R
- added SW1: SW_SPDT, SamacSys_Parts:EG1215AA, symbol Switch:SW_SPDT
- added U8: REF5025ID, Package_SO:SOIC-8_3.9x4.9mm_P1.27mm, symbol Reference_Voltage:REF5025ID
- added U9: LT3032-3.3, Package_DFN_QFN:Linear_DE14MA, symbol Regulator_Linear:LT3032-3.3
- C44: renamed from C5; footprint Capacitor_SMD:C_0805_2012Metric_Pad1.15x1.40mm_HandSolder -> Capacitor_SMD:C_0603_1608Metric_Pad1.05x0.95mm_HandSolder
- C46: renamed from C8; value C 68u -> C 47u
- R24: renamed from R67; footprint Resistor_SMD:R_1206_3216Metric_Pad1.42x1.75mm_HandSolder -> Resistor_SMD:R_0805_2012Metric_Pad1.15x1.40mm_HandSolder
- R25: renamed from R66; footprint Resistor_SMD:R_1206_3216Metric_Pad1.42x1.75mm_HandSolder -> Resistor_SMD:R_0805_2012Metric_Pad1.15x1.40mm_HandSolder
- R26: renamed from R13; value R -> R 51k
- R27: renamed from R14; value R -> R 25.5k
- renumbered C7 to C30, C1 to C31, C6 to C35, C2 to C39, C3 to C43, C9 to C45, C4 to C47, D3 to D2, D1 to D3, D5 to D4, D4 to D5, J4 to J1, R11 to R18, R12 to R19, R9 to R22, R10 to R23, U2 to U10, U3 to U11, U4 to U12, U1 to U7
Connections:
- net +5V: now also C32.1, C38.1, R20.1, U8.2 (Vin), U9.12 (~SHDNP), U9.14 (INP); no longer U10.7 (FB)
- net +BATT: now also SW1.1 (A)
- net -5V: now also C42.1, U9.10 (~SHDNN), U9.6 (INN), U9.9 (INN)
- net GND: now also C32.2, C33.2, C34.2, C37.2, C38.2, C41.2, C42.2, R21.2, SW1.3 (C), U8.4 (GND), U9.4 (GND), U9.5 (GND); no longer H1.1, H2.1, H3.1, H4.1
- net Pwr1: now also SW1.2 (B)
- new net: R20.2, R21.1, U10.7 (FB)
- new net: C34.1, U8.5 (Trim/NR)
- new net: C36.2, U9.3 (BYPP)
- new net: C40.2, U9.11 (BYPN)
- new net +2V5: C33.1, U8.6 (Vout)
- new net +3.3VADC: C36.1, C37.1, U9.1 (OUTP)
- new net -3V3: C40.1, C41.1, U9.7 (OUTN)
- no-connect marks 5 -> 9
Other:
- note added: "When fix 5v option is used leave FB resistor to ground open and place 0 ohm resistor to output"
