File: Building sensor/Designs/EMI_sensor_control_Rev2.0/file5D43B07A.sch (KiCad schematic (older format))
At the start: 46 parts, among them U8 AD8021ARZ, U9 AD7763BSVZ

Commit message: overdue backup
Parts:
- removed C17, C25, C26, C27, C28, C29, C30, C31, C33, C34: C 100n, Capacitor_SMD:C_0603_1608Metric_Pad1.05x0.95mm_HandSolder, symbol Device:C
- removed C18: C 33p, Capacitor_SMD:C_0402_1005Metric, symbol Device:C
- removed C19: C 100u, Capacitor_Tantalum_SMD:CP_EIA-7343-30_AVX-N_Pad2.25x2.55mm_HandSolder, symbol Device:C
- removed C21, C32: C 10n, Capacitor_SMD:C_0805_2012Metric_Pad1.15x1.40mm_HandSolder, symbol Device:C
- removed FB1, FB10, FB2, FB3, FB4, FB5, FB6, FB7, FB8, FB9: Ferrite_Bead, Capacitor_SMD:C_0603_1608Metric_Pad1.05x0.95mm_HandSolder, symbol Device:Ferrite_Bead
- removed L2: L 8.2n, Inductor_SMD:L_0603_1608Metric_Pad1.05x0.95mm_HandSolder, symbol Device:L
- removed R18, R65: R 10k, Resistor_SMD:R_1206_3216Metric_Pad1.42x1.75mm_HandSolder, symbol Device:R
- removed R20: R 100, Resistor_SMD:R_1206_3216Metric_Pad1.42x1.75mm_HandSolder, symbol Device:R
- removed R21: R 160k, Resistor_SMD:R_1206_3216Metric_Pad1.42x1.75mm_HandSolder, symbol Device:R
- removed R22, R30: R 10, Resistor_SMD:R_1206_3216Metric_Pad1.42x1.75mm_HandSolder, symbol Device:R
- removed R24, R25: R 18, Resistor_SMD:R_0805_2012Metric_Pad1.15x1.40mm_HandSolder, symbol Device:R
- removed U9: AD7763BSVZ, footprints:AD7763BSVZ, symbol 2019-07-11_15-43-26:AD7763BSVZ
Connections:
- net labels removed: +2V5, ADCReset, ADCSync, ADR0b, ADR1b, ADR2b, AGND1b, AGND2b, AGND3b, AGND4b, DRDY, FSI, FSOb, GNDD, GNDREF, GNDS, MCLK, Pin12b, Pin14b, Pin15b, Pin24b, Pin27b, Pin33b, Pin41b, Pin44b, Pin4b, Pin63b, Pin6b, SCO, SDI, SDLb, SDO, SH0b, SH1, SH2, Vref4.1
- wire segments 262 -> 51

Commit message: backup
2/04/2020
Parts:
- added C? (x7): C 1u, Capacitor_SMD:C_0402_1005Metric, symbol Device:C
- added R? (x4): R 100k, Resistor_SMD:R_0805_2012Metric_Pad1.15x1.40mm_HandSolder, symbol Device:R
- added U?: ADS127L01IPBSR, PBS0032A_N, symbol 2019-12-03_16-41-56:ADS127L01IPBSR
Connections:
- net GND: now also C?.1, C?.1, C?.1, C?.1, C?.1, C?.1, C?.2, R?.1, R?.2, R?.2, U?.26 (DGND), U?.32 (AVDD), U?.5 (AGND)
- new net: C?.1, U?.1 (LVDD)
- new net: R?.2, U?.18 (DAISYIN)
- new net: C?.2, U?.25 (CAP3)
- new net: C?.2, U?.11 (CAP2)
- new net: C?.2, U?.2 (CAP1)
- new net: R?.1, U?.30 (FORMAT)
- new net: R?.1, U?.29 (HR)
- new net: R?.1, U?.14 (FSMODE)
- new net +3V0: C?.2, C?.2, U?.27 (DVDD), U?.31 (AGND)
- new net +3V3: C?.2, R?.2, U?.6 (AVDD)
- new net ADC_Reset: U?.28 (RESET_PWDN_N)
- new net Bx_CS: U?.23 (CS_N)
- new net Bx_Clk: U?.22 (SCLK)
- new net Bx_FIL0: U?.13 (FILTER0)
- new net Bx_FIL1: U?.12 (FILTER1)
- new net Bx_MISO: U?.20 (DOUT)
- new net Bx_MOSI: U?.21 (DIN)
- new net Bx_N: U?.3 (AINN)
- new net Bx_OSR0: U?.16 (OSR0)
- new net Bx_OSR1: U?.15 (OSR1)
- new net Bx_P: U?.4 (AINP)
- new net Bx_START: U?.17 (START)

Commit message: Back up
Backup of rev 2.0 for board
Parts:
- removed C22: C 5.6p, Capacitor_SMD:C_0402_1005Metric, symbol Device:C
- removed C23, C24: C 33p, Capacitor_SMD:C_0402_1005Metric, symbol Device:C
- removed R26, R27: R 1k, Resistor_SMD:R_0805_2012Metric_Pad1.15x1.40mm_HandSolder, symbol Device:R
- removed R28, R29: R 649, Resistor_SMD:R_0805_2012Metric_Pad1.15x1.40mm_HandSolder, symbol Device:R
- added C?: C 1u, Capacitor_SMD:C_0402_1005Metric, symbol Device:C
- added R? (x2): R 1k, Resistor_SMD:R_0805_2012Metric_Pad1.15x1.40mm_HandSolder, symbol Device:R
- added R? (x2): R 10k, Resistor_SMD:R_0805_2012Metric_Pad1.15x1.40mm_HandSolder, symbol Device:R
Connections:
- net +3V0: now also C?.2, U?.32 (AVDD), U?.6 (AVDD); no longer C?.2, U?.27 (DVDD), U?.31 (AGND)
- net +3V3: now also C?.2, U?.27 (DVDD); no longer C?.2, U?.6 (AVDD)
- net BxFiltered: now also R?.2
- net GND: now also U?.10 (REFN), U?.31 (AGND), C?.2, R?.1, R?.1; no longer U?.32 (AVDD)
- net -BxFiltered: now reaches R23.1, U8.6 (VOUT)
- net -BxFiltered: now also R?.2
- net at U?.7 (REXT): now also R?.2
- net at U?.8 (INTLDO_N): now also R?.2
- net +2V5: now reaches U?.9 (REFP)
- net +2V5: now also C?.1
- net Bx_N: no longer names the net of U?.3 (AINN)
- net Bx_N: now also R?.1
- net Bx_P: no longer names the net of U?.4 (AINP)
- net Bx_P: now also R?.1

Commit message: Rev 2.0 Complete
Rev 2.0 of PCB Completed
SCHM, PCB layout, and gerber files generated
Parts:
- added C57: C 270p, Capacitor_SMD:C_0603_1608Metric_Pad1.05x0.95mm_HandSolder, symbol Device:C
- added C58, C63: C 1u, Capacitor_SMD:C_0805_2012Metric_Pad1.15x1.40mm_HandSolder, symbol Device:C
- added C59: C 470p, Capacitor_SMD:C_0603_1608Metric_Pad1.05x0.95mm_HandSolder, symbol Device:C
- added C60: C 1n, Capacitor_SMD:C_0603_1608Metric_Pad1.05x0.95mm_HandSolder, symbol Device:C
- added C61: C 22n, Capacitor_SMD:C_0805_2012Metric_Pad1.15x1.40mm_HandSolder, symbol Device:C
- added C64: C 270p, Capacitor_SMD:C_0805_2012Metric_Pad1.15x1.40mm_HandSolder, symbol Device:C
- added R32: R 200 1%, Resistor_SMD:R_0805_2012Metric_Pad1.15x1.40mm_HandSolder, symbol Device:R
- added R37, R49: R 1.2K 1%, Resistor_SMD:R_0805_2012Metric_Pad1.15x1.40mm_HandSolder, symbol Device:R
- added R40, R45: R 1.2k 1%, Resistor_SMD:R_0805_2012Metric_Pad1.15x1.40mm_HandSolder, symbol Device:R
- added R41, R46: R 330 1%, Resistor_SMD:R_0805_2012Metric_Pad1.15x1.40mm_HandSolder, symbol Device:R
- added R42, R47: R 4.99 1%, Resistor_SMD:R_0805_2012Metric_Pad1.15x1.40mm_HandSolder, symbol Device:R
- added R43, R48: R 10 1%, Resistor_SMD:R_0805_2012Metric_Pad1.15x1.40mm_HandSolder, symbol Device:R
- added U15: THS4551IDGKR, Package_SO:VSSOP-8_3.0x3.0mm_P0.65mm, symbol THS4551IDGKR:THS4551IDGKR
- C49, C50, C51, C52, C53, C54, C55, C56: renamed from C?; footprint Capacitor_SMD:C_0402_1005Metric -> Capacitor_SMD:C_0805_2012Metric_Pad1.15x1.40mm_HandSolder
- C62: renamed from C20; footprint Capacitor_SMD:C_0805_2012Metric_Pad1.15x1.40mm_HandSolder -> Capacitor_SMD:C_0603_1608Metric_Pad1.05x0.95mm_HandSolder
- R38: renamed from R23; value R 2k -> R 2k 1%
- R39: renamed from R17; value R 2k -> R 2k 1%
- R44: renamed from R19; value R 1k -> R 1k 1%
- U13: renamed from U?; footprint PBS0032A_N -> SamacSys_Parts:QFP50P700X700X120-32N
- U14: renamed from U8; footprint footprints:AD8021ARZ -> Package_SO:SOIC-8_3.9x4.9mm_P1.27mm
- gave numbers to parts that had none: 8
Connections:
- net -BxFiltered: now also R45.1; no longer R31.2
- net BxFiltered: now also R40.1; no longer R30.2
- net GND: now also C58.1, C63.1, U15.6 (VS-)
- net Bx_DRDY: now reaches U13.19 (DRDY_FSYNC_N)
- net at U13.24 (CLK): now also R32.1
- new net: C60.1, C64.1, R46.2, U15.1 (IN-)
- new net: C63.2, U15.2 (VOCM)
- new net: C57.1, R42.1, U15.4 (OUT+)
- new net: C64.2, R47.1, U15.5 (OUT-)
- new net: C57.2, C60.2, R41.2, U15.8 (IN+)
- new net: C59.2, R37.1, R40.2, R41.1
- new net: C59.1, R45.2, R46.1, R49.2
- new net: R37.2, R42.2, R43.1
- new net: R47.2, R48.1, R49.1
- new net +3.3VADC: C58.2, U15.3 (VS+), U15.7 (~PD~)
- new net ADC_CLK: R32.2
- new net AINN_Bx: C61.1, R31.2, R48.2
- new net AINP_Bx: C61.2, R30.2, R43.2
Other:
- moved on the sheet: C62, R38, R39, R44, U14
